File: electrical/camper_van.kicad_sch (KiCad schematic)
At the start: 32 parts, among them J1 Starter Battery, J2 Ignition, J3 Input Flow Sensor, J4 Output Flow Sensor, J5 Input Flow Sensor, J6 Output Flow Sensor, J7 Battery Box, J8 Battery Box, J9 Duoetto Remote, K1 Relay 200A, K2 Relay 200A, K3 Relay 250A, K4 Relay 250A, M1 Battery Box Fan, U1 Input Flow Sensor, U2 Output Flow Sensor, U3 DS18B20

Commit message: lots of redesign
Connections:
- net at F3.1, K1.11: no longer J7.7 (Pin_7)
- net at F4.2, F6.1, Renogy 200Ah2.1 (+): now also J7.8 (Pin_8); no longer J7.10 (Pin_10)
- net at F3.2, F5.1, Renogy 200Ah1.1 (+): now also J7.7 (Pin_7); no longer J7.9 (Pin_9)
- net at F4.1, K2.11: no longer J7.8 (Pin_8)
- net +5V renamed VCC_3V3
- net Management Module/5V renamed Management Module/3V3
- net Management Module/Battery 1 In Sensor: no longer names the net of J8.9 (Pin_9)
- net Management Module/Battery 2 In Sensor: no longer names the net of J8.10 (Pin_10)
- no-connect marks 0 -> 4
Other:
- sheet Management Module ports: added 3V3; removed 5V, Battery 1 In Sensor, Battery 2 In Sensor

Commit message: work in progress
Parts:
- K1, K2: value Relay 200A -> Relay 120A
Connections:
- net GND: no longer K3.A2, K4.A2
- net at J7.10 (Pin_10): now also J7.9 (Pin_9), K3.A2, K4.A2
- net Management Module/Vin: now reaches J8.10 (Pin_10)
- net Management Module/Vin: now also J8.9 (Pin_9)
- net Fuse and Switch Module/Solar Charge Battery 2 renamed Management Module/Solar Charge Battery 2
- net Management Module/Battery 1 Out Sensor renamed Management Module/Battery 1 Fuse Sensor
- net Management Module/Battery 2 Out Sensor renamed Management Module/Battery 2 Fuse Sensor
- no-connect marks 4 -> 5
Other:
- sheet Fuse and Switch Module ports: added Air Suspension On/Off, Battery 2 SW, Fridge On/Off, Inverter On/Off, Lights & Aux On/Off, Power On/Off SW, Pump On/Off, Solar Charge Battery 2 SW; removed Battery 2, Power On/Off A, Power On/Off B, Solar Charge Battery 2
- sheet Management Module ports: added Battery 1 Fuse Sensor, Battery 2 Fuse Sensor, Battery 2 SW, Power On/Off SW, Solar Charge Battery 2 SW, Vin; removed Battery 1 Out Sensor, Battery 2, Battery 2 Out Sensor, Power On/Off A, Power On/Off B
- moved on the sheet: Duoetto_Heater1, J9

Commit message: UPdated
Parts:
- removed J7: Battery Box, symbol Connector:Conn_01x16_Socket
- removed J8: Battery Box, Connector_Molex:Molex_Mini-Fit_Jr_5569-16A2_2x08_P4.20mm_Horizontal, symbol Connector:Conn_01x16_Pin
- added F10, F11, F12, F13, F14, F15: 10A, symbol Device:Fuse
- added F16, F17: 15A, symbol Device:Fuse
- added F7: ANL 50A, symbol Device:Fuse
- added F8: ANL 250A, symbol Device:Fuse
- added F9: 5A, symbol Device:Fuse
- added Inverter1: ~, symbol camper_van:Inverter
- added J10, J17: Fan, symbol Connector:Conn_01x02_Pin
- added J11, J16: Fan, symbol Connector:Conn_01x02_Socket
- added J12: Temp, symbol Connector:Conn_01x03_Pin
- added J13: Temp, symbol Connector:Conn_01x03_Socket
- added J14: Battery & Fuse, symbol Connector:Conn_01x04_Pin
- added J15: Battery & Fuse, symbol Connector:Conn_01x04_Socket
- added J18: Inverter remote, symbol Connector:Conn_01x02_Pin
- added J19: Relays, symbol Connector:Conn_01x04_Socket
- added J2, J27: Solar Panel 2, symbol Connector:Conn_01x02_Socket
- added J20: 12V Power, symbol Connector:Conn_01x02_Socket
- added J21: Relays, symbol Connector:Conn_01x04_Pin
- added J22: Battery 2, symbol Connector:Conn_01x04_Socket
- added J23: 12V Power, symbol Connector:Conn_01x02_Pin
- added J25: Inverter Remote, symbol Connector:Conn_01x02_Socket
- added J26: Solar Panel 1, symbol Connector:Conn_01x02_Socket
- added J28: Solar Charge, symbol Connector:Conn_01x02_Pin
- added J29: Battery 2, symbol Connector:Conn_01x04_Pin
- added J30: Solar Panel 1, symbol Connector:Conn_01x02_Pin
- added J31: Solar Panel 2, symbol Connector:Conn_01x02_Pin
- added J8: RS485, symbol Connector:Conn_01x02_Pin
- added J9: RS485, symbol Connector:Conn_01x02_Socket
- added SW1: 12V Power On/Off, symbol Switch:SW_SPST
- added SW10: Solar Panel 1, symbol Switch:SW_SPST
- added SW11: Solar Panel 2, symbol Switch:SW_SPST
- added SW12: Solar Chg Battery 2, symbol Switch:SW_SPST
- added SW13: Battery 2 On/Off, symbol Switch:SW_SPST
- added SW2: Inverter, symbol Switch:SW_SPST
- added SW3: Hot Water, symbol Switch:SW_SPST
- added SW4: Air Suspension, symbol Switch:SW_SPST
- added SW5: Pump, symbol Switch:SW_SPST
- added SW6: Fridge, symbol Switch:SW_SPST
- added SW7: Lights, symbol Switch:SW_SPST
- added SW8, SW9: Aux, symbol Switch:SW_SPST
- J6: renamed from J5; footprint Connector_Molex:CONN_SD-172648-0000_02_MOL -> (none)
- J7: renamed from J6; footprint Connector_Molex:CONN_SD-172648-0000_02_MOL -> (none)
- renumbered J9 to J24, J2 to J3, J3 to J4, J4 to J5, SC2 to SC1, SC1 to SC2
Connections:
- net +12V: now also F10.2, F11.2, F12.2, F13.2, F14.2, F15.2, F7.1, F8.1, F9.2, J20.2 (Pin_2), J23.2 (Pin_2), SW12.1 (A)
- net Fuse and Switch Module/Duoetto 12V: now also F7.2
- net GND: now also Inverter1.5 (GND), J10.2 (Pin_2), J11.2 (Pin_2), J12.3 (Pin_3), J13.3 (Pin_3), J16.1 (Pin_1), J2.2 (Pin_2), J20.1 (Pin_1), J22.4 (Pin_4), J23.1 (Pin_1), J26.2 (Pin_2), J27.2 (Pin_2), J28.2 (Pin_2), J29.4 (Pin_4), J30.2 (Pin_2), J31.2 (Pin_2), SW13.1 (A)
- net Management Module/3V3: now also J13.1 (Pin_1)
- net Management Module/Battery 1 Fuse Sensor: now also J15.3 (Pin_3)
- net Management Module/Battery 1 Relay: now also J19.3 (Pin_3)
- net Management Module/Battery 1 Vin: now also J15.1 (Pin_1)
- net Management Module/Battery 2 Fuse Sensor: now also J15.4 (Pin_4)
- net Management Module/Battery 2 Relay: now also J19.4 (Pin_4)
- net Management Module/Battery 2 Vin: now also J15.2 (Pin_2)
- net Management Module/Battery Box Fan: now also J11.1 (Pin_1)
- net Management Module/Solar Charge Battery 2: now also J19.1 (Pin_1)
- net Management Module/Temperature Sensors: now also J13.2 (Pin_2)
- net Management Module/Vin: now also J19.2 (Pin_2)
- net RS485 Rx: now also J9.2 (Pin_2)
- net RS485 Tx: now also J9.1 (Pin_1)
- net VCC_3V3: now also J12.1 (Pin_1)
- net at F5.2, K3.13: now also J14.3 (Pin_3)
- net at K3.A1: now also J21.3 (Pin_3)
- net at K3.A2, K4.A2: now also J21.2 (Pin_2)
- net at M1.1 (+): now also J10.1 (Pin_1)
- net at K1.A1, K2.A1: now also J21.1 (Pin_1)
- net at F4.2, F6.1, Renogy 200Ah2.1 (+): now also J14.2 (Pin_2)
- net at F6.2, K4.13: now also J14.4 (Pin_4)
- net at DC-DC 20A1.3 (A): now also J8.2 (Pin_2)
- net at DC-DC 20A1.4 (B): now also J8.1 (Pin_1)
- net at F3.2, F5.1, Renogy 200Ah1.1 (+): now also J14.1 (Pin_1)
- net at K4.A1: now also J21.4 (Pin_4)
- net at U3.2 (DQ): now also J12.2 (Pin_2)
- net Fuse and Switch Module/Duoetto Power On/Off renamed Fuse and Switch Module/Duoetto Power SW
- net Fuse and Switch Module/Duoetto Power SW: now also SW3.1 (A)
- net Fuse and Switch Module/Solar 1: no longer names the net of SC1.1 (+)
- net Fuse and Switch Module/Solar 1: now also J31.1 (Pin_1)
- net Fuse and Switch Module/Solar 2: no longer names the net of SC2.1 (+)
- net Fuse and Switch Module/Solar 2: now also J30.1 (Pin_1)
- net Solar Charge: no longer names the net of DC-DC 50A MPPT1.1 (Solar)
- net Solar Charge: now also J2.1 (Pin_1)
- new net: Inverter1.2 (A), J25.1 (Pin_1)
- new net: Inverter1.3 (B), J25.2 (Pin_2)
- new net: F17.1, J27.1 (Pin_1)
- new net: J29.2 (Pin_2), SW12.2 (B)
- new net: J29.3 (Pin_3), SW13.2 (B)
- new net: F16.2, SW10.2 (B)
- new net: J18.2 (Pin_2), SW2.1 (A)
- new net: J18.1 (Pin_1), SW2.2 (B)
- new net: F17.2, SW11.2 (B)
- new net: J17.1 (Pin_1), SW1.1 (A)
- new net: J17.2 (Pin_2), SW1.2 (B)
- new net: F16.1, J26.1 (Pin_1)
- new net Fuse and Switch Module/Air Suspension SW: SW4.1 (A)
- new net Fuse and Switch Module/Air Suspension SW Fuse: F10.1, SW4.2 (B)
- new net Fuse and Switch Module/Aux SW: SW8.1 (A)
- new net Fuse and Switch Module/Aux SW Fuse: F14.1, SW8.2 (B)
- new net Fuse and Switch Module/Duoetto Power SW Fuse: F9.1, SW3.2 (B)
- new net Fuse and Switch Module/Fridge SW: SW6.1 (A)
- new net Fuse and Switch Module/Fridge SW Fuse: F12.1, SW6.2 (B)
- new net Fuse and Switch Module/Inverter: F8.2, Inverter1.4 (12V)
- new net Fuse and Switch Module/Lights SW: SW7.1 (A)
- new net Fuse and Switch Module/Lights SW Fuse: F13.1, SW7.2 (B)
- new net Fuse and Switch Module/Pump SW: SW5.1 (A)
- new net Fuse and Switch Module/Pump SW Fuse: F11.1, SW5.2 (B)
- new net Fuse and Switch Module/Solar: J28.1 (Pin_1), SW10.1 (A), SW11.1 (A)
- new net Fuse and Switch Module/Spare SW: SW9.1 (A)
- new net Fuse and Switch Module/Spare SW Fuse: F15.1, SW9.2 (B)
- new net Management Module/Battery 2 SW: J22.1 (Pin_1)
- new net Management Module/Power On/Off SW: J16.2 (Pin_2)
- new net Management Module/Solar Charge Battery 2 SW: J22.3 (Pin_3)
- new net VIN: J22.2 (Pin_2), J29.1 (Pin_1)
- no-connect marks 5 -> 0
Other:
- sheet Fuse and Switch Module ports: added Air Suspension SW, Air Suspension SW Fuse, Aux SW, Aux SW Fuse, Duoetto Power SW, Duoetto Power SW Fuse, Fridge SW, Fridge SW Fuse, Inverter, Lights SW, Lights SW Fuse, Pump SW, Pump SW Fuse, Solar, Spare SW, Spare SW Fuse; removed Air Suspension On/Off, Battery 2 SW, Duoetto Power On/Off, Fridge On/Off, Inverter On/Off, Lights & Aux On/Off, Power On/Off SW, Pump On/Off, RS485 Rx, RS485 Tx, Solar 1, Solar 2, Solar Charge, Solar Charge Battery 2 SW
- note added: "Control Panel"
- note added: "Fuse Box"
- note added: "Internal Switch Panel"
- moved on the sheet: DC-DC 50A MPPT1, Duoetto_Heater1, F1, F3, F4, F5, F6, J24, J4, J5, J6, J7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

Commit message: First attempt at PCB design
Parts:
- removed J10: Fan, symbol Connector:Conn_01x02_Pin
- removed J11: Fan, symbol Connector:Conn_01x02_Socket
- removed M1: Battery Box Fan, symbol Motor:Fan
- added J10: Fans, symbol Connector:Conn_01x04_Pin
- added J11: Fans, symbol Connector:Conn_01x04_Socket
- added J24: Lights, symbol Connector:Conn_01x02_Socket
- added J25: Lights, Connector_Molex:Molex_Mini-Fit_Jr_5569-02A1_2x01_P4.20mm_Horizontal, symbol Connector:Conn_01x02_Pin
- added J26: Duoetto Remote, Connector_Molex:Molex_Mini-Fit_Jr_5569-02A1_2x01_P4.20mm_Horizontal, symbol Connector:Conn_01x02_Pin
- added LA1: Lamp, symbol Device:Lamp
- added M1: Fan1, symbol Motor:Fan_4pin
- added M2: Fan2, symbol Motor:Fan_4pin
- J16, J17: value Fan -> Power On/Off
- renumbered J4 to J1, J5 to J2, J24 to J27, J25 to J28, J26 to J29, J1 to J3, J27 to J30, J28 to J31, J29 to J32, J30 to J33, J31 to J34, J6 to J4, J7 to J5, J2 to J6, J3 to J7
Connections:
- net +12V: now also M1.2 (+), M2.2 (+)
- net Fuse and Switch Module/Duoetto Power SW: no longer Duoetto_Heater1.1 (Pwr)
- net GND: now also J25.2 (Pin_2), M1.1 (-), M2.1 (-)
- new net: J24.1 (Pin_1), LA1.2 (+)
- new net: J24.2 (Pin_2), LA1.1 (-)
- new net: J10.1 (Pin_1), M1.4 (PWM)
- new net: J10.2 (Pin_2), M1.3 (Tacho)
- new net: J10.3 (Pin_3), M2.4 (PWM)
- new net: J10.4 (Pin_4), M2.3 (Tacho)
- new net Fuse and Switch Module/Duoetto Pwr: Duoetto_Heater1.1 (Pwr)
- new net Fuse and Switch Module/Lights: J25.1 (Pin_1)
- new net Fuse and Switch Module/RS485 Rx: J26.1 (Pin_1)
- new net Fuse and Switch Module/RS485 Tx: J26.2 (Pin_2)
- new net Management Module/Battery Box Fan1 Control: J11.1 (Pin_1)
- new net Management Module/Battery Box Fan1 Sensor: J11.2 (Pin_2)
- new net Management Module/Battery Box Fan2 Control: J11.3 (Pin_3)
- new net Management Module/Battery Box Fan2 Sensor: J11.4 (Pin_4)
Other:
- sheet Fuse and Switch Module ports: added Duoetto Pwr, Lights, RS485 Rx, RS485 Tx; removed none
- sheet Management Module ports: added Battery Box Fan1 Control, Battery Box Fan1 Sensor, Battery Box Fan2 Control, Battery Box Fan2 Sensor; removed Battery Box Fan
- moved on the sheet: A1, DC-DC 20A1, DC-DC 50A MPPT1, Duoetto_Heater1, F1, F10, F11, F12, F13, F14, F15, F16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
