File: electrical/display.kicad_sch (KiCad schematic)
At the start: 7 parts, among them U14 IPS 3.5" Display, U16 BA00

Commit message: lots of redesign
Parts:
- C47: renamed from C30; value 0.1uF -> 22uF
- R95: renamed from R94; value 71k5 -> 68k
- R96: renamed from R95; value 71k5 -> 10k
- renumbered A3 to A4, C29 to C46, U16 to U25, U14 to U26
Connections:
- net VCC_D renamed VCC_D_9V5
Changed lines of the file:
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@@
 		(dnp no)
 		(fields_autoplaced yes)
-		(property "Reference" "#PWR0146"
+		(property "Reference" "#PWR0184"
 			(at 67.31 48.26 0)
 			(effects
@@
 			(project "camper_van"
 				(path "/e095b45b-2ed6-497c-8100-020e1086a4e5/91acac86-faa4-4d81-9e47-c92be50b558f"
-					(reference "#PWR0146")
+					(reference "#PWR0184")
 					(unit 1)
 				)
@@
 		(dnp no)
 		(fields_autoplaced yes)
-		(property "Reference" "#PWR091"
+		(property "Reference" "#PWR0182"
 			(at 29.21 40.64 0)
 			(effects
@@
 			(project "camper_van"
 				(path "/e095b45b-2ed6-497c-8100-020e1086a4e5/91acac86-faa4-4d81-9e47-c92be50b558f"
-					(reference "#PWR091")
+					(reference "#PWR0182")
 					(unit 1)
 				)
@@
 		(dnp no)
 		(fields_autoplaced yes)
-		(property "Reference" "R95"
+		(property "Reference" "R96"
 			(at 69.85 36.8299 0)
 			(effects
@@
 			)
 		)
-		(property "Value" "71k5"
+		(property "Value" "10k"
 			(at 69.85 39.3699 0)
 			(effects
@@
 			)
 		)
+		(property "Sim.Type" ""
+			(at 67.31 38.1 0)
+			(effects
+				(font
+					(size 1.27 1.27)
+				)
+				(hide yes)
+			)
+		)
 		(pin "2"
 		)
@@
 			(project "camper_van"
 				(path "/e095b45b-2ed6-497c-8100-020e1086a4e5/91acac86-faa4-4d81-9e47-c92be50b558f"
-					(reference "R95")
+					(reference "R96")
 					(unit 1)
 				)
@@
 		(dnp no)
 		(fields_autoplaced yes)
-		(property "Reference" "#PWR0145"
+		(property "Reference" "#PWR0183"
 			(at 50.8 45.72 0)
 			(effects
@@
 			(project "camper_van"
 				(path "/e095b45b-2ed6-497c-8100-020e1086a4e5/91acac86-faa4-4d81-9e47-c92be50b558f"
-					(reference "#PWR0145")
+					(reference "#PWR0183")
 					(unit 1)
 				)
@@
 		(dnp no)
 		(fields_autoplaced yes)
-		(property "Reference" "#PWR088"
+		(property "Reference" "#PWR0181"
 			(at 29.21 27.94 0)
 			(effects
@@
 			(project "camper_van"
 				(path "/e095b45b-2ed6-497c-8100-020e1086a4e5/91acac86-faa4-4d81-9e47-c92be50b558f"
-					(reference "#PWR088")
+					(reference "#PWR0181")
 					(unit 1)
 				)
@@
 		(dnp no)
 		(fields_autoplaced yes)
-		(property "Reference" "C30"
+		(property "Reference" "C47"
 			(at 80.01 27.5081 0)
 			(effects
@@
 			)
 		)
-		(property "Value" "0.1uF"
+		(property "Value" "22uF"
 			(at 80.01 30.0481 0)
 			(effects
@@
 			)
 		)
+		(property "Sim.Type" ""
+			(at 77.47 29.21 0)
+			(effects
+				(font
+					(size 1.27 1.27)
+				)
+				(hide yes)
+			)
+		)
 		(pin "1"
 		)
@@
 			(project "camper_van"
 				(path "/e095b45b-2ed6-497c-8100-020e1086a4e5/91acac86-faa4-4d81-9e47-c92be50b558f"
-					(reference "C30")
+					(reference "C47")
 					(unit 1)
 				)
@@
 		(dnp no)
 		(fields_autoplaced yes)
-		(property "Reference" "C29"
+		(property "Reference" "C46"
 			(at 31.75 28.7781 0)
 			(effects
@@
 			)
 		)
+		(property "Sim.Type" ""
+			(at 29.21 30.48 0)
+			(effects
+				(font
+					(size 1.27 1.27)
+				)
+				(hide yes)
+			)
+		)
 		(pin "1"
 		)
@@
 			(project "camper_van"
 				(path "/e095b45b-2ed6-497c-8100-020e1086a4e5/91acac86-faa4-4d81-9e47-c92be50b558f"
-					(reference "C29")
+					(reference "C46")
 					(unit 1)
 				)
@@
 		(dnp no)
 		(fields_autoplaced yes)
-		(property "Reference" "#PWR0122"
+		(property "Reference" "#PWR0187"
 			(at 93.98 123.19 0)
 			(effects
@@
 			(project "camper_van"
 				(path "/e095b45b-2ed6-497c-8100-020e1086a4e5/91acac86-faa4-4d81-9e47-c92be50b558f"
-					(reference "#PWR0122")
+					(reference "#PWR0187")
 					(unit 1)
 				)
@@
 		(dnp no)
 		(fields_autoplaced yes)
-		(property "Reference" "#PWR0116"
+		(property "Reference" "#PWR0188"
 			(at 154.94 62.23 0)
 			(effects
@@
 			)
 		)
-		(property "Value" "VCC_D"
+		(property "Value" "VCC_D_9V5"
 			(at 154.94 53.34 0)
 			(effects
@@
 			(project "camper_van"
 				(path "/e095b45b-2ed6-497c-8100-020e1086a4e5/91acac86-faa4-4d81-9e47-c92be50b558f"
-					(reference "#PWR0116")
+					(reference "#PWR0188")
 					(unit 1)
 				)
@@
 		(dnp no)
 		(fields_autoplaced yes)
-		(property "Reference" "U16"
+		(property "Reference" "U25"
 			(at 50.8 20.32 0)
 			(effects
@@
 			)
 		)
+		(property "Sim.Type" ""
+			(at 50.8 29.21 0)
+			(effects
+				(font
+					(size 1.27 1.27)
+				)
+				(hide yes)
+			)
+		)
 		(pin "2"
 		)
@@
 			(project "camper_van"
 				(path "/e095b45b-2ed6-497c-8100-020e1086a4e5/91acac86-faa4-4d81-9e47-c92be50b558f"
-					(reference "U16")
+					(reference "U25")
 					(unit 1)
 				)
@@
 		(dnp no)
 		(fields_autoplaced yes)
-		(property "Reference" "#PWR0147"
+		(property "Reference" "#PWR0185"
 			(at 77.47 26.67 0)
 			(effects
@@
 			)
 		)
-		(property "Value" "VCC_D"
+		(property "Value" "VCC_D_9V5"
 			(at 77.47 17.78 0)
 			(effects
@@
 			(project "camper_van"
 				(path "/e095b45b-2ed6-497c-8100-020e1086a4e5/91acac86-faa4-4d81-9e47-c92be50b558f"
-					(reference "#PWR0147")
+					(reference "#PWR0185")
 					(unit 1)
 				)
@@
 		(dnp no)
 		(fields_autoplaced yes)
-		(property "Reference" "#PWR0124"
+		(property "Reference" "#PWR0189"
 			(at 157.48 118.11 0)
 			(effects
@@
 			(project "camper_van"
 				(path "/e095b45b-2ed6-497c-8100-020e1086a4e5/91acac86-faa4-4d81-9e47-c92be50b558f"
-					(reference "#PWR0124")
+					(reference "#PWR0189")
 					(unit 1)
 				)
@@
 		(dnp no)
 		(fields_autoplaced yes)
-		(property "Reference" "#PWR0148"
+		(property "Reference" "#PWR0186"
 			(at 77.47 39.37 0)
 			(effects
@@
 			(project "camper_van"
 				(path "/e095b45b-2ed6-497c-8100-020e1086a4e5/91acac86-faa4-4d81-9e47-c92be50b558f"
-					(reference "#PWR0148")
+					(reference "#PWR0186")
 					(unit 1)
 				)
@@
 		(dnp no)
 		(fields_autoplaced yes)
-		(property "Reference" "U14"
+		(property "Reference" "U26"
 			(at 96.1233 81.28 0)
 			(effects
@@
 			)
 		)
+		(property "Sim.Type" ""
+			(at 93.98 99.06 0)
+			(effects
+				(font
+					(size 1.27 1.27)
+				)
+				(hide yes)
+			)
+		)
 		(pin "10"
 		)
@@
 			(project "camper_van"
 				(path "/e095b45b-2ed6-497c-8100-020e1086a4e5/91acac86-faa4-4d81-9e47-c92be50b558f"
-					(reference "U14")
+					(reference "U26")
 					(unit 1)
 				)
@@
 		(dnp no)
 		(fields_autoplaced yes)
-		(property "Reference" "A3"
+		(property "Reference" "A4"
 			(at 162.1633 109.22 0)
 			(effects
@@
 			)
 		)
+		(property "Sim.Type" ""
+			(at 157.48 83.82 0)
+			(effects
+				(font
+					(size 1.27 1.27)
+				)
+				(hide yes)
+			)
+		)
 		(pin "30"
 		)
@@
 			(project "camper_van"
 				(path "/e095b45b-2ed6-497c-8100-020e1086a4e5/91acac86-faa4-4d81-9e47-c92be50b558f"
-					(reference "A3")
+					(reference "A4")
 					(unit 1)
 				)
@@
 		(dnp no)
 		(fields_autoplaced yes)
-		(property "Reference" "R94"
+		(property "Reference" "R95"
 			(at 69.85 29.2099 0)
 			(effects
@@
 			)
 		)
-		(property "Value" "71k5"
+		(property "Value" "68k"
 			(at 69.85 31.7499 0)
 			(effects
@@
 			)
 		)
+		(property "Sim.Type" ""
+			(at 67.31 30.48 0)
+			(effects
+				(font
+					(size 1.27 1.27)
+				)
+				(hide yes)
+			)
+		)
 		(pin "2"
 		)
@@
 			(project "camper_van"
 				(path "/e095b45b-2ed6-497c-8100-020e1086a4e5/91acac86-faa4-4d81-9e47-c92be50b558f"
-					(reference "R94")
-					(unit 1)
-				)
+					(reference "R95")
+					(unit 1)
+				)

Commit message: work in progress
Parts:
- renumbered C46 to C54, C47 to C55, R95 to R103, R96 to R104, U25 to U24, U26 to U25
Changed lines of the file:
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@@
 		(dnp no)
 		(fields_autoplaced yes)
-		(property "Reference" "#PWR0184"
+		(property "Reference" "#PWR0187"
 			(at 67.31 48.26 0)
 			(effects
@@
 			(project "camper_van"
 				(path "/e095b45b-2ed6-497c-8100-020e1086a4e5/91acac86-faa4-4d81-9e47-c92be50b558f"
-					(reference "#PWR0184")
+					(reference "#PWR0187")
 					(unit 1)
 				)
@@
 		(dnp no)
 		(fields_autoplaced yes)
-		(property "Reference" "#PWR0182"
+		(property "Reference" "#PWR0185"
 			(at 29.21 40.64 0)
 			(effects
@@
 			(project "camper_van"
 				(path "/e095b45b-2ed6-497c-8100-020e1086a4e5/91acac86-faa4-4d81-9e47-c92be50b558f"
-					(reference "#PWR0182")
+					(reference "#PWR0185")
 					(unit 1)
 				)
@@
 		(dnp no)
 		(fields_autoplaced yes)
-		(property "Reference" "R96"
+		(property "Reference" "R104"
 			(at 69.85 36.8299 0)
 			(effects
@@
 			(project "camper_van"
 				(path "/e095b45b-2ed6-497c-8100-020e1086a4e5/91acac86-faa4-4d81-9e47-c92be50b558f"
-					(reference "R96")
+					(reference "R104")
 					(unit 1)
 				)
@@
 		(dnp no)
 		(fields_autoplaced yes)
-		(property "Reference" "#PWR0183"
+		(property "Reference" "#PWR0186"
 			(at 50.8 45.72 0)
 			(effects
@@
 			(project "camper_van"
 				(path "/e095b45b-2ed6-497c-8100-020e1086a4e5/91acac86-faa4-4d81-9e47-c92be50b558f"
-					(reference "#PWR0183")
+					(reference "#PWR0186")
 					(unit 1)
 				)
@@
 		(dnp no)
 		(fields_autoplaced yes)
-		(property "Reference" "#PWR0181"
+		(property "Reference" "#PWR0184"
 			(at 29.21 27.94 0)
 			(effects
@@
 			(project "camper_van"
 				(path "/e095b45b-2ed6-497c-8100-020e1086a4e5/91acac86-faa4-4d81-9e47-c92be50b558f"
-					(reference "#PWR0181")
+					(reference "#PWR0184")
 					(unit 1)
 				)
@@
 		(dnp no)
 		(fields_autoplaced yes)
-		(property "Reference" "C47"
+		(property "Reference" "C55"
 			(at 80.01 27.5081 0)
 			(effects
@@
 			(project "camper_van"
 				(path "/e095b45b-2ed6-497c-8100-020e1086a4e5/91acac86-faa4-4d81-9e47-c92be50b558f"
-					(reference "C47")
+					(reference "C55")
 					(unit 1)
 				)
@@
 		(dnp no)
 		(fields_autoplaced yes)
-		(property "Reference" "C46"
+		(property "Reference" "C54"
 			(at 31.75 28.7781 0)
 			(effects
@@
 			(project "camper_van"
 				(path "/e095b45b-2ed6-497c-8100-020e1086a4e5/91acac86-faa4-4d81-9e47-c92be50b558f"
-					(reference "C46")
+					(reference "C54")
 					(unit 1)
 				)
@@
 		(dnp no)
 		(fields_autoplaced yes)
-		(property "Reference" "#PWR0187"
+		(property "Reference" "#PWR0190"
 			(at 93.98 123.19 0)
 			(effects
@@
 			(project "camper_van"
 				(path "/e095b45b-2ed6-497c-8100-020e1086a4e5/91acac86-faa4-4d81-9e47-c92be50b558f"
-					(reference "#PWR0187")
+					(reference "#PWR0190")
 					(unit 1)
 				)
@@
 		(dnp no)
 		(fields_autoplaced yes)
-		(property "Reference" "#PWR0188"
+		(property "Reference" "#PWR0191"
 			(at 154.94 62.23 0)
 			(effects
@@
 			(project "camper_van"
 				(path "/e095b45b-2ed6-497c-8100-020e1086a4e5/91acac86-faa4-4d81-9e47-c92be50b558f"
-					(reference "#PWR0188")
+					(reference "#PWR0191")
 					(unit 1)
 				)
@@
 		(dnp no)
 		(fields_autoplaced yes)
-		(property "Reference" "U25"
+		(property "Reference" "U24"
 			(at 50.8 20.32 0)
 			(effects
@@
 			(project "camper_van"
 				(path "/e095b45b-2ed6-497c-8100-020e1086a4e5/91acac86-faa4-4d81-9e47-c92be50b558f"
-					(reference "U25")
+					(reference "U24")
 					(unit 1)
 				)
@@
 		(dnp no)
 		(fields_autoplaced yes)
-		(property "Reference" "#PWR0185"
+		(property "Reference" "#PWR0188"
 			(at 77.47 26.67 0)
 			(effects
@@
 			(project "camper_van"
 				(path "/e095b45b-2ed6-497c-8100-020e1086a4e5/91acac86-faa4-4d81-9e47-c92be50b558f"
-					(reference "#PWR0185")
+					(reference "#PWR0188")
 					(unit 1)
 				)
@@
 		(dnp no)
 		(fields_autoplaced yes)
-		(property "Reference" "#PWR0189"
+		(property "Reference" "#PWR0192"
 			(at 157.48 118.11 0)
 			(effects
@@
 			(project "camper_van"
 				(path "/e095b45b-2ed6-497c-8100-020e1086a4e5/91acac86-faa4-4d81-9e47-c92be50b558f"
-					(reference "#PWR0189")
+					(reference "#PWR0192")
 					(unit 1)
 				)
@@
 		(dnp no)
 		(fields_autoplaced yes)
-		(property "Reference" "#PWR0186"
+		(property "Reference" "#PWR0189"
 			(at 77.47 39.37 0)
 			(effects
@@
 			(project "camper_van"
 				(path "/e095b45b-2ed6-497c-8100-020e1086a4e5/91acac86-faa4-4d81-9e47-c92be50b558f"
-					(reference "#PWR0186")
+					(reference "#PWR0189")
 					(unit 1)
 				)
@@
 		(dnp no)
 		(fields_autoplaced yes)
-		(property "Reference" "U26"
+		(property "Reference" "U25"
 			(at 96.1233 81.28 0)
 			(effects
@@
 			(project "camper_van"
 				(path "/e095b45b-2ed6-497c-8100-020e1086a4e5/91acac86-faa4-4d81-9e47-c92be50b558f"
-					(reference "U26")
+					(reference "U25")
 					(unit 1)
 				)
@@
 		(dnp no)
 		(fields_autoplaced yes)
-		(property "Reference" "R95"
+		(property "Reference" "R103"
 			(at 69.85 29.2099 0)
 			(effects
@@
 			(project "camper_van"
 				(path "/e095b45b-2ed6-497c-8100-020e1086a4e5/91acac86-faa4-4d81-9e47-c92be50b558f"
-					(reference "R95")
-					(unit 1)
-				)
+					(reference "R103")
+					(unit 1)
+				)

Commit message: UPdated
Parts:
- removed A4: Arduino_Nano_v3.x, Module:Arduino_Nano, symbol MCU_Module:Arduino_Nano_v3.x
- removed U25: IPS 3.5" Display, Display:CR2013-MI2120, symbol camper_van:Display IPS 3.5{dblquote}
- added A4: Arduino_Nano_ESP32, Module:Arduino_Nano, symbol MCU_Module:Arduino_Nano_ESP32
- added C44: 0.33uF, symbol Device:C_Polarized_Small_US
- added C45: 0.1uF, Capacitor_THT:CP_Radial_Tantal_D5.0mm_P5.00mm, symbol Device:C_Polarized_Small_US
- added U27: LM7805, Package_TO_SOT_THT:TO-220-3_Vertical, symbol Regulator_Linear:LM7805_TO220
- added U28: IPS 3.5" Display, Display:CR2013-MI2120, symbol camper_van:Display IPS 3.5{dblquote}
- renumbered C54 to C42, C55 to C43, R103 to R82, R104 to R83, U24 to U26
Connections:
- net CTP_SCL: now also A4.24 (SCL/A5), U28.10 (CTP_SCL)
- net CTP_SDA: now also A4.23 (SDA/A4), U28.12 (CTP_SDA)
- net GND: now also A4.29 (GND), A4.4 (GND), C44.2, C45.2, U27.2 (GND), U28.2 (GND)
- net RS485 Rx: now also A4.2 (D0/RX)
- net RS485 Tx: now also A4.1 (D1/TX)
- net VCC_D_9V5: now also A4.30 (VIN)
- new net: A4.6 (D3), U28.3 (~{CS})
- new net: A4.7 (D4), U28.4 (RESET)
- new net: A4.8 (D5), U28.5 (D/~{C})
- new net: A4.14 (D11/COPI), U28.6 (MOSI)
- new net: A4.16 (D13/SCK), U28.7 (SCK)
- new net: A4.9 (D6), U28.8 (LED)
- new net: A4.15 (D12/CIPO), U28.9 (MISO)
- new net CTP_INT: A4.11 (D8), U28.13 (CTP_INT)
- new net CTP_RST: A4.10 (D7), U28.11 (CTP_RST)
- new net SD_CS: A4.12 (D9), U28.14 (SD_CS)
- new net VCC_5V: C45.1, U27.3 (VO), U28.1 (VCC)
- new net VCC_MM_9V5: C44.1, U27.1 (VI)
- no-connect marks 26 -> 13

Commit message: First attempt at PCB design
Parts:
- renumbered C42 to C49, C43 to C50, C44 to C51, C45 to C52, R82 to R65, R83 to R66, U26 to U29, U27 to U30, U28 to U31
Connections:
- net SD_CS: now also A4.13 (D10/CS); no longer A4.12 (D9)
Changed lines of the file:
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@@
+	)
+	(no_connect
+		(at 130.81 105.41)
 	)
 	(no_connect
@@
 		(at 95.25 77.47)
 	)
-	(no_connect
-		(at 130.81 107.95)
-	)
 	(wire
 		(pts
@@
 	(wire
 		(pts
-			(xy 133.35 105.41) (xy 130.81 105.41)
-		)
-		(stroke
-			(width 0)
-			(type default)
-		)
-	)
-	(wire
-		(pts
 			(xy 130.81 82.55) (xy 144.78 82.55)
+		)
+		(stroke
+			(width 0)
+			(type default)
+		)
+	)
+	(wire
+		(pts
+			(xy 130.81 107.95) (xy 133.35 107.95)
 		)
 		(stroke
@@
 	)
 	(label "SD_CS"
-		(at 133.35 105.41 0)
+		(at 133.35 107.95 0)
 		(effects
 			(font
@@
 		(dnp no)
 		(fields_autoplaced yes)
-		(property "Reference" "#PWR0224"
+		(property "Reference" "#PWR0201"
 			(at 67.31 48.26 0)
 			(effects
@@
 			(project "camper_van"
 				(path "/e095b45b-2ed6-497c-8100-020e1086a4e5/91acac86-faa4-4d81-9e47-c92be50b558f"
-					(reference "#PWR0224")
+					(reference "#PWR0201")
 					(unit 1)
 				)
@@
 		(dnp no)
 		(fields_autoplaced yes)
-		(property "Reference" "#PWR0228"
+		(property "Reference" "#PWR0205"
 			(at 101.6 41.91 0)
 			(effects
@@
 			(project "camper_van"
 				(path "/e095b45b-2ed6-497c-8100-020e1086a4e5/91acac86-faa4-4d81-9e47-c92be50b558f"
-					(reference "#PWR0228")
+					(reference "#PWR0205")
 					(unit 1)
 				)
@@
 		(dnp no)
 		(fields_autoplaced yes)
-		(property "Reference" "#PWR0222"
+		(property "Reference" "#PWR0199"
 			(at 29.21 40.64 0)
 			(effects
@@
 			(project "camper_van"
 				(path "/e095b45b-2ed6-497c-8100-020e1086a4e5/91acac86-faa4-4d81-9e47-c92be50b558f"
-					(reference "#PWR0222")
+					(reference "#PWR0199")
 					(unit 1)
 				)
@@
 		(dnp no)
 		(fields_autoplaced yes)
-		(property "Reference" "R83"
+		(property "Reference" "R66"
 			(at 69.85 36.8299 0)
 			(effects
@@
 			(project "camper_van"
 				(path "/e095b45b-2ed6-497c-8100-020e1086a4e5/91acac86-faa4-4d81-9e47-c92be50b558f"
-					(reference "R83")
+					(reference "R66")
 					(unit 1)
 				)
@@
 		(dnp no)
 		(fields_autoplaced yes)
-		(property "Reference" "#PWR0223"
+		(property "Reference" "#PWR0200"
 			(at 50.8 45.72 0)
 			(effects
@@
 			(project "camper_van"
 				(path "/e095b45b-2ed6-497c-8100-020e1086a4e5/91acac86-faa4-4d81-9e47-c92be50b558f"
-					(reference "#PWR0223")
+					(reference "#PWR0200")
 					(unit 1)
 				)
@@
 		(on_board yes)
 		(dnp no)
-		(property "Reference" "#PWR0234"
+		(property "Reference" "#PWR0211"
 			(at 181.61 96.52 0)
 			(effects
@@
 			(project "camper_van"
 				(path "/e095b45b-2ed6-497c-8100-020e1086a4e5/91acac86-faa4-4d81-9e47-c92be50b558f"
-					(reference "#PWR0234")
+					(reference "#PWR0211")
 					(unit 1)
 				)
@@
 		(dnp no)
 		(fields_autoplaced yes)
-		(property "Reference" "#PWR0221"
+		(property "Reference" "#PWR0198"
 			(at 29.21 27.94 0)
 			(effects
@@
 			(project "camper_van"
 				(path "/e095b45b-2ed6-497c-8100-020e1086a4e5/91acac86-faa4-4d81-9e47-c92be50b558f"
-					(reference "#PWR0221")
+					(reference "#PWR0198")
 					(unit 1)
 				)
@@
 		(dnp no)
 		(fields_autoplaced yes)
-		(property "Reference" "C43"
+		(property "Reference" "C50"
 			(at 80.01 27.5081 0)
 			(effects
@@
 			(project "camper_van"
 				(path "/e095b45b-2ed6-497c-8100-020e1086a4e5/91acac86-faa4-4d81-9e47-c92be50b558f"
-					(reference "C43")
+					(reference "C50")
 					(unit 1)
 				)
@@
 		(dnp no)
 		(fields_autoplaced yes)
-		(property "Reference" "U28"
+		(property "Reference" "U31"
 			(at 179.4667 95.25 0)
 			(effects
@@
 			(project "camper_van"
 				(path "/e095b45b-2ed6-497c-8100-020e1086a4e5/91acac86-faa4-4d81-9e47-c92be50b558f"
-					(reference "U28")
+					(reference "U31")
 					(unit 1)
 				)
@@
 		(dnp no)
 		(fields_autoplaced yes)
-		(property "Reference" "#PWR0232"
+		(property "Reference" "#PWR0209"
 			(at 134.62 78.74 0)
 			(effects
@@
 			(project "camper_van"
 				(path "/e095b45b-2ed6-497c-8100-020e1086a4e5/91acac86-faa4-4d81-9e47-c92be50b558f"
-					(reference "#PWR0232")
+					(reference "#PWR0209")
 					(unit 1)
 				)
@@
 		(dnp no)
 		(fields_autoplaced yes)
-		(property "Reference" "C42"
+		(property "Reference" "C49"
 			(at 31.75 28.7781 0)
 			(effects
@@
 			(project "camper_van"
 				(path "/e095b45b-2ed6-497c-8100-020e1086a4e5/91acac86-faa4-4d81-9e47-c92be50b558f"
-					(reference "C42")
+					(reference "C49")
 					(unit 1)
 				)
@@
 		(dnp no)
 		(fields_autoplaced yes)
-		(property "Reference" "C45"
+		(property "Reference" "C52"
 			(at 129.54 30.0481 0)
 			(effects
@@
 			(project "camper_van"
 				(path "/e095b45b-2ed6-497c-8100-020e1086a4e5/91acac86-faa4-4d81-9e47-c92be50b558f"
-					(reference "C45")
+					(reference "C52")
 					(unit 1)
 				)
@@
 		(dnp no)
 		(fields_autoplaced yes)
-		(property "Reference" "U26"
+		(property "Reference" "U29"
 			(at 50.8 20.32 0)
 			(effects
@@
 			(project "camper_van"
 				(path "/e095b45b-2ed6-497c-8100-020e1086a4e5/91acac86-faa4-4d81-9e47-c92be50b558f"
-					(reference "U26")
+					(reference "U29")
 					(unit 1)
 				)
@@
 		(dnp no)
 		(fields_autoplaced yes)
-		(property "Reference" "#PWR0225"
+		(property "Reference" "#PWR0202"
 			(at 77.47 26.67 0)
 			(effects
@@
 			(project "camper_van"
 				(path "/e095b45b-2ed6-497c-8100-020e1086a4e5/91acac86-faa4-4d81-9e47-c92be50b558f"
-					(reference "#PWR0225")
+					(reference "#PWR0202")
 					(unit 1)
 				)
@@
 		(dnp no)
 		(fields_autoplaced yes)
-		(property "Reference" "#PWR0226"
+		(property "Reference" "#PWR0203"
 			(at 77.47 39.37 0)
 			(effects
@@
 			(project "camper_van"
 				(path "/e095b45b-2ed6-497c-8100-020e1086a4e5/91acac86-faa4-4d81-9e47-c92be50b558f"
-					(reference "#PWR0226")
+					(reference "#PWR0203")
 					(unit 1)
 				)
@@
 		(dnp no)
 		(fields_autoplaced yes)
-		(property "Reference" "#PWR0235"
+		(property "Reference" "#PWR0212"
 			(at 181.61 137.16 0)
 			(effects
@@
 			(project "camper_van"
 				(path "/e095b45b-2ed6-497c-8100-020e1086a4e5/91acac86-faa4-4d81-9e47-c92be50b558f"
-					(reference "#PWR0235")
+					(reference "#PWR0212")
 					(unit 1)
 				)
@@
 		(dnp no)
 		(fields_autoplaced yes)
-		(property "Reference" "#PWR0230"
+		(property "Reference" "#PWR0207"
 			(at 116.84 41.91 0)
 			(effects
@@
 			(project "camper_van"
 				(path "/e095b45b-2ed6-497c-8100-020e1086a4e5/91acac86-faa4-4d81-9e47-c92be50b558f"
-					(reference "#PWR0230")
+					(reference "#PWR0207")
 					(unit 1)
 				)
@@
 		(on_board yes)
 		(dnp no)
-		(property "Reference" "#PWR0233"
+		(property "Reference" "#PWR0210"
 			(at 135.89 31.75 0)
 			(effects
@@
 			(project "camper_van"
 				(path "/e095b45b-2ed6-497c-8100-020e1086a4e5/91acac86-faa4-4d81-9e47-c92be50b558f"
-					(reference "#PWR0233")
+					(reference "#PWR0210")
 					(unit 1)
 				)
@@
 		(dnp no)
 		(fields_autoplaced yes)
-		(property "Reference" "#PWR0231"
+		(property "Reference" "#PWR0208"
 			(at 127 41.91 0)
 			(effects
@@
 			(project "camper_van"
 				(path "/e095b45b-2ed6-497c-8100-020e1086a4e5/91acac86-faa4-4d81-9e47-c92be50b558f"
-					(reference "#PWR0231")
+					(reference "#PWR0208")
 					(unit 1)
 				)
@@
 		(dnp no)
 		(fields_autoplaced yes)
-		(property "Reference" "C44"
+		(property "Reference" "C51"
 			(at 104.14 30.0481 0)
 			(effects
@@
 			(project "camper_van"
 				(path "/e095b45b-2ed6-497c-8100-020e1086a4e5/91acac86-faa4-4d81-9e47-c92be50b558f"
-					(reference "C44")
+					(reference "C51")
 					(unit 1)
 				)
@@
 		(dnp no)
 		(fields_autoplaced yes)
-		(property "Reference" "#PWR0227"
+		(property "Reference" "#PWR0204"
 			(at 101.6 29.21 0)
 			(effects
@@
 			(project "camper_van"
 				(path "/e095b45b-2ed6-497c-8100-020e1086a4e5/91acac86-faa4-4d81-9e47-c92be50b558f"
-					(reference "#PWR0227")
+					(reference "#PWR0204")
 					(unit 1)
 				)
@@
 		(dnp no)
 		(fields_autoplaced yes)
-		(property "Reference" "U27"
+		(property "Reference" "U30"
 			(at 116.84 21.59 0)
 			(effects
@@
 			(project "camper_van"
 				(path "/e095b45b-2ed6-497c-8100-020e1086a4e5/91acac86-faa4-4d81-9e47-c92be50b558f"
-					(reference "U27")
+					(reference "U30")
 					(unit 1)
 				)
@@
 		(dnp no)
 		(fields_autoplaced yes)
-		(property "Reference" "R82"
+		(property "Reference" "R65"
 			(at 69.85 29.2099 0)
 			(effects
@@
 			(project "camper_van"
 				(path "/e095b45b-2ed6-497c-8100-020e1086a4e5/91acac86-faa4-4d81-9e47-c92be50b558f"
-					(reference "R82")
+					(reference "R65")
 					(unit 1)
 				)
@@
 		(dnp no)
 		(fields_autoplaced yes)
-		(property "Reference" "#PWR0229"
+		(property "Reference" "#PWR0206"
 			(at 113.03 129.54 0)
 			(effects
@@
 			(project "camper_van"
 				(path "/e095b45b-2ed6-497c-8100-020e1086a4e5/91acac86-faa4-4d81-9e47-c92be50b558f"
-					(reference "#PWR0229")
+					(reference "#PWR0206")
 					(unit 1)
 				)
