File: electrical/fuse_switch.kicad_sch (KiCad schematic)
At the start: 90 parts, among them J18 Power, J19 Fuse and Switch Box, J20 Solar Panel 1, J21 Solar Panel 2, J22 Power, SW10 Solar Panel 1, SW11 Solar Panel 2, SW2 12V Power On/Off, SW3 Battery 2 On/Off, SW4 Solar/50A charge Battery 2, SW5 Inverter, SW6 Pump, SW7 Fridge, SW8 Lights & Aux, SW9 Hot Water, U11 BA00, U12 MCP6004, U15 MCP6004

Commit message: lots of redesign
Parts:
- added C24, C28: 1uF, symbol Device:C
- added C25, C26, C27, C29, C30, C31, C32, C33: 100nF, symbol Device:C_Small
- C23: renamed from C14; value 0.1uF -> 22uF
- R52: renamed from R88; value 71k5 -> 68k
- R53: renamed from R89; value 71k5 -> 10k
- renumbered A4 to A3, C13 to C22, C27 to C34, C25 to C35, C28 to C36, C26 to C37, C15 to C38, C16 to C39, C17 to C40, C18 to C41, C19 to C42, C20 to C43, C21 to C44, C22 to C45, D12 to D9, F12 to F10, F8 to F11, F9 to F12, F10 to F13, F7 to F14, F13 to F7, F14 to F8, F11 to F9, J22 to J19, J19 to J22, R85 to R47, R86 to R48, R83 to R49, R84 to R50, R90 to R51, R68 to R54, R69 to R55, R81 to R58, R66 to R59, R82 to R60, R67 to R61, R55 to R62, R87 to R63, R54 to R64, R79 to R65, R74 to R66, R46 to R67, R47 to R68, R48 to R69, R49 to R70, R58 to R71, R59 to R72, R60 to R73, R61 to R74, R50 to R75, R51 to R76, R62 to R77, R63 to R78, R52 to R79, R53 to R80, R64 to R81, R65 to R82, R80 to R83, R91 to R84, R92 to R85, R93 to R86, R75 to R87, R76 to R88, R77 to R89, R78 to R90, R70 to R91, R71 to R92, R72 to R93, R73 to R94, SW7 to SW10, SW8 to SW11, SW10 to SW2, SW11 to SW3, SW2 to SW4, SW3 to SW5, SW4 to SW6, SW9 to SW7, SW5 to SW8, SW6 to SW9, U15 to U22, U11 to U23, U12 to U24
Connections:
- net GND: no longer C36.2, C37.2, C39.2, C41.2, C43.2, C45.2, R48.2, R50.2, R55.2, R57.2, R68.2, R70.2, R72.2, R74.2, U22.11 (V-), U24.11 (V-)
- net at A3.22 (A3), C40.2, R69.1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: now also C29.1
- net at A3.26 (A7), C44.2, R73.1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: now also C33.1
- net at A3.21 (A2), C38.2, R67.1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: now also C31.1
- net at A3.19 (A0), C34.2, R54.1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: now also C26.1, C27.1
- net at A3.25 (A6), C42.2, R71.1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: now also C32.1
- net +5V_FS renamed VCC_3V3_FS
- net VCC_3V3_FS: no longer U22.4 (V+), U24.4 (V+)
- net VCC_FS renamed VCC_FS_9V5
- new net GNDA: C24.2, C25.2, C28.2, C30.2, C36.2, C37.2, C39.2, C41.2, C43.2, C45.2, R48.2, R50.2, R55.2, R57.2, R68.2, R70.2, R72.2, R74.2, U22.11 (V-), U24.11 (V-)
- new net GNDD: C26.2, C27.2, C29.2, C31.2, C32.2, C33.2
- new net VCC_3V3: C24.1, C25.1, C28.1, C30.1, U22.4 (V+), U24.4 (V+)
Other:
- moved on the sheet: U22E

Commit message: work in progress
Parts:
- removed J18, J19: Power, symbol Connector:Conn_01x02_Socket
- removed J22: Fuse and Switch Box, symbol Connector:Conn_01x06_Socket
- removed R47, R48, R49, R50: 10k, symbol Device:R
- added C38, C39, C40, C41: 1uF, symbol Device:C
- added C44, C45: 100nF, symbol Device:C_Small
- added F10: 50A, symbol Device:Fuse
- added F12: 10A, symbol Device:Fuse
- added J20: Conn_01x06_Socket, symbol Connector:Conn_01x06_Socket
- added R53, R55: 5k9, symbol Device:R
- added R54, R56, R68, R70, R74: 10k, symbol Device:R
- added R59, R60, R63, R64: 154k, symbol Device:R
- added R67: 35.7K 1%, Resistor_THT:R_Axial_DIN0207_L6.3mm_D2.5mm_P10.16mm_Horizontal, symbol Device:R
- added R72: 6k2, symbol Device:R
- added SW8: Air Suspension, symbol Switch:SW_SPST
- F13: renamed from F14; value 250A -> ANL 250A
- F7, F8: value 20A -> 15A
- F9: value 50A -> ANL 50A
- renumbered C22 to C24, C23 to C25, C24 to C26, C25 to C27, C26 to C28, C27 to C29, C28 to C30, C32 to C31, C30 to C32, C31 to C42, C29 to C43, C38 to C46, C39 to C47, C40 to C48, C41 to C49, C42 to C50, C43 to C51, C44 to C52, C45 to C53, F10 to F11, F11 to F14, F12 to F15, F13 to F16, J20 to J18, J21 to J19, R92 to R100, R93 to R101, R94 to R102, R51 to R46, R52 to R47, R53 to R48, R54 to R49, R55 to R50, R56 to R51, R57 to R52, R58 to R57, R59 to R58, R60 to R61, R61 to R62, R62 to R65, R63 to R66, R64 to R69, R65 to R71, R66 to R73, R67 to R75, R68 to R76, R69 to R77, R70 to R78, R71 to R79, R72 to R80, R73 to R81, R74 to R82, R75 to R83, R76 to R84, R77 to R85, R78 to R86, R79 to R87, R80 to R88, R81 to R89, R82 to R90, R83 to R91, R84 to R92, R85 to R93, R86 to R94, R87 to R95, R88 to R96, R89 to R97, R90 to R98, R91 to R99, SW9 to SW10, SW10 to SW11, SW11 to SW12, SW8 to SW9, U23 to U21, U24 to U22, U22 to U23
Connections:
- net Power On/Off B is gone; now on net GND: SW4.2 (B)
- net +12V: now also SW6.2 (B), F10.1, F12.1, J20.2 (Pin_2), R74.1
- net GND: now also J20.6 (Pin_6), R68.2, R70.2; no longer SW6.2 (B)
- net GNDA: now also C40.2, C41.2, R54.2, R56.2
- net GNDD: now also C44.2, C45.2
- net VIN: now also J20.4 (Pin_4)
- net Fridge On/Off: now reaches R89.1, R93.1, R97.2, SW11.2 (B)
- net at U23.12 (+): now also C41.1, R60.2
- net at U23.13 (-): now also R55.2, R56.1; no longer U23.14
- net Lights & Aux On/Off: now reaches R90.1, R94.1, R98.2, SW12.2 (B)
- net at C52.2, R81.1, U22.14: now also A3.24 (A5), C45.1; no longer A3.26 (A7), C33.1
- net Pump On/Off: now reaches R88.1, R92.1, R96.2, SW10.2 (B)
- net at U23.10 (+): now also C40.1, R59.2
- net at U23.8: now also A3.25 (A6), C29.1, C38.2, R53.1; no longer U23.9 (-)
- net at A3.19 (A0), C34.2, R49.1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: now also C31.1; no longer C28.1, C29.1
- net at A3.20 (A1), C35.2, R51.1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: now also C33.1
- net Inverter On/Off: now reaches R87.1, R91.1, R95.2, SW9.2 (B)
- net at C50.2, R79.1, U22.8: now also A3.23 (A4), C44.1; no longer A3.25 (A6), C31.1
- net Battery 2 renamed Battery 2 SW
- net Battery 2 SW: now also J20.3 (Pin_3)
- net Power On/Off A renamed Power On/Off SW
- net Power On/Off SW: now also J20.1 (Pin_1)
- net Solar Charge Battery 2 renamed Solar Charge Battery 2 SW
- net Solar Charge Battery 2 SW: now also J20.5 (Pin_5)
- new net: A3.26 (A7), C28.1, C39.2, R55.1, U23.14
- new net: C39.1, R60.1, R64.2
- new net: F12.2, R72.1, R74.2, SW8.1 (A)
- new net: C38.1, R59.1, R63.2
- new net: R53.2, R54.1, U23.9 (-)
- new net: F10.2, R67.1
- new net: R64.1, R67.2, R68.1
- new net Air Suspension On/Off: R63.1, R70.1, R72.2, SW8.2 (B)
- no-connect marks 17 -> 15
Other:
- note added: "Air Suspension Switch and Fuse Sensor"
- note added: "Spare Fuse Sensor"
- moved on the sheet: C28, C29, C31, C33, C42, C43, F11, F14, F15, F16, SW4, SW5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

Commit message: UPdated
Parts:
- removed A3: Arduino_Nano_v3.x, Module:Arduino_Nano, symbol MCU_Module:Arduino_Nano_v3.x
- removed C26, C30, C34, C35, C36, C37, C38, C39, C40, C41, C46, C47, C48, C49, C50, C51, C52, C53: 1uF, symbol Device:C
- removed C42, C43, C44, C45: 100nF, symbol Device:C_Small
- removed F10: 50A, symbol Device:Fuse
- removed F11: 5A, symbol Device:Fuse
- removed F12, F14: 10A, symbol Device:Fuse
- removed F13: ANL 250A, symbol Device:Fuse
- removed F15, F7, F8: 15A, symbol Device:Fuse
- removed F16: Fuse, symbol Device:Fuse
- removed F9: ANL 50A, symbol Device:Fuse
- removed J18: Solar Panel 1, symbol Connector:Conn_01x02_Socket
- removed J19: Solar Panel 2, symbol Connector:Conn_01x02_Socket
- removed J20: Conn_01x06_Socket, symbol Connector:Conn_01x06_Socket
- removed R100, R101, R102, R82, R91, R92, R93, R94, R99: 10k, symbol Device:R
- removed R49: 5k9, symbol Device:R
- removed R83, R84, R85, R86, R87, R88, R89, R90: 154k, symbol Device:R
- removed R95, R96, R97, R98: 6k2, symbol Device:R
- removed SW10: Pump, symbol Switch:SW_SPST
- removed SW11: Fridge, symbol Switch:SW_SPST
- removed SW12: Lights & Aux, symbol Switch:SW_SPST
- removed SW2: Solar Panel 1, symbol Switch:SW_SPST
- removed SW3: Solar Panel 2, symbol Switch:SW_SPST
- removed SW4: 12V Power On/Off, symbol Switch:SW_SPST
- removed SW5: Battery 2 On/Off, symbol Switch:SW_SPST
- removed SW6: Solar/50A charge Battery 2, symbol Switch:SW_SPST
- removed SW7: Hot Water, symbol Switch:SW_SPST
- removed SW8: Air Suspension, symbol Switch:SW_SPST
- removed SW9: Inverter, symbol Switch:SW_SPST
- removed U22, U23: MCP6004, symbol Amplifier_Operational:MCP6004
- added A3: Arduino_Nano_ESP32, Module:Arduino_Nano, symbol MCU_Module:Arduino_Nano_ESP32
- added C26, C30, C34, C35, C36, C37, C38, C39, C40, C41: 100nF, symbol Device:C_Small
- added SW15: SW_Push, symbol Switch:SW_Push
- added U22, U23, U24, U25: ILQ615-3, symbol camper_van:ILQ615-3
- R50, R52, R54, R68, R69, R70, R76, R78: value 10k -> 680
- R51, R53, R77: value 5k9 -> 680
- R55, R75, R79, R81: value 5k9 -> 1k2
- R56, R66, R73, R74, R80: value 10k -> 1k2
- R57, R58, R59, R64: value 154k -> 1k2
- R60, R61, R62, R63: value 154k -> 680
- R65, R67: value 35.7K 1% -> 1k2; footprint Resistor_THT:R_Axial_DIN0207_L6.3mm_D2.5mm_P10.16mm_Horizontal -> (none)
- R71: value 6k2 -> 680
- R72: value 6k2 -> 1k2
- renumbered R46 to R47, R47 to R48, R48 to R49
Connections:
- net Duoetto 12V: now also R59.2; no longer R65.1
- net GND: now also U22.2, U22.3, U22.6, U22.7, U23.2, U23.3, U23.6, U23.7, U24.2, U24.3, U24.6, U24.7, U25.2, U25.3, U25.6, U25.7; no longer R66.2, R68.2, R69.2, R70.2
- net GNDD: now also C27.2, C32.2, R50.2, R51.2, R52.2, R53.2, R54.2, R60.2, R61.2, R62.2, R63.2, R68.2, R69.2, R70.2, R71.2, R76.2, R77.2, R78.2, A3.29 (GND), A3.4 (GND), C26.2, C30.2, C34.2, C35.2, C36.2, C37.2, C38.2, C39.2, C40.2, C41.2, SW15.2
- net VCC_3V3: now also U22.10, U22.11, U22.14, U22.15, U23.10, U23.11, U23.14, U23.15, U24.10, U24.11, U24.14, U24.15, U25.10, U25.11, U25.14, U25.15; no longer C27.1, C32.1
- net VCC_FS_9V5: now also A3.30 (VIN)
- net Switch Lights: now reaches R78.1
- net Switch Lights: now also A3.20 (A1), C41.1, U25.9; no longer R77.2
- net Switch Fridge: now reaches R77.1
- net Switch Fridge: now also A3.15 (D12/CIPO), C40.1, U25.13
- net Fridge SW Fuse: now reaches R73.2
- net Fridge SW Fuse: no longer R71.1
- net Duoetto Power SW Fuse: now reaches R58.2
- net at R56.1: now also U23.1; no longer R55.2
- net at R55.1: now also U22.1; no longer C28.1
- net Duoetto Power SW: now reaches R64.2
- net Duoetto Power SW: no longer R60.1
- net Spare SW Fuse: now reaches R57.2
- net at R57.1: now also U22.5; no longer R61.2
- net at R79.1: now also U23.8
- net at R75.1: now also U24.8
- net at R81.1: now also U25.8
- net at R72.1: now also U23.5; no longer R74.2
- net at R59.1: now also U24.5; no longer R63.2
- net Lights SW: now reaches R81.2
- net Fuse Duoetto Pwr: now reaches C29.1, R53.1
- net Fuse Duoetto Pwr: now also A3.8 (D5), U24.16
- net Fuse Duoetto 12V: now reaches R54.1
- net Fuse Duoetto 12V: now also A3.6 (D3), C30.1, U24.12; no longer R53.2
- net Inverter: now reaches R75.2
- net Inverter: no longer R76.1
- net at R80.1: now also U25.4; no longer R79.2
- net at R67.1: now also U22.8
- net Switch Duoetto Pwr: now reaches C31.1
- net Switch Duoetto Pwr: now also R60.1, A3.9 (D6), U24.13
- net Fuse_Air: now reaches R50.1
- net Fuse_Air: now also A3.12 (D9), C26.1, U22.16
- net at D9.1 (K), R47.1: now also A3.25 (A6)
- net at R58.1: now also U24.1; no longer R62.2
- net Fuse Aux: now reaches R51.1
- net Fuse Aux: now also C27.1, A3.21 (A2), U23.16; no longer C33.1
- net Fuse Spare: now reaches R52.1
- net Fuse Spare: now also C28.1, A3.23 (SDA/A4), U22.12; no longer R51.2
- net +12V: no longer names the net of R73.1
- net +12V: now also U25.1; no longer R74.1
- removed net Air Suspension On/Off: R63.1, R70.1, R72.2
- removed net Duoetto Power On/Off: R61.1, R69.1, R71.2
- removed net GNDA: C27.2, C32.2, R50.2, R52.2, R54.2, R56.2, R76.2, R78.2, R80.2
- net Solar Charge renamed Solar
- new net: A3.3 (~{RESET}), SW15.1
- new net: R65.1, U22.4
- new net: R64.1, U24.4
- new net: R66.1, U23.4
- new net: R74.1, U25.5
- new net Air Suspension SW: R65.2
- new net Air Suspension SW Fuse: R55.2
- new net Aux SW: R66.2
- new net Aux SW Fuse: R56.2
- new net Fridge SW: R80.2
- new net Fuse Fridge: A3.14 (D11/COPI), C36.1, R69.1, U25.16
- new net Fuse Inverter: A3.7 (D4), C38.1, R71.1, U24.9
- new net Fuse Lights: A3.19 (A0), C37.1, R70.1, U25.12
- new net Fuse Pump: A3.10 (D7), C35.1, R68.1, U23.12
- new net Lights SW Fuse: R74.2
- new net Pump SW: R79.2
- new net Pump SW Fuse: R72.2
- new net Spare SW: R67.2
- new net Switch Aux: A3.22 (A3), C33.1, R62.1, U23.13
- new net Switch Pump: A3.11 (D8), C39.1, R76.1, U23.9
- new net Switch Spare: A3.24 (SCL/A5), C34.1, R63.1, U22.9
- new net Switch_Air: A3.13 (D10/CS), C32.1, R61.1, U22.13
- no-connect marks 15 -> 9
Other:
- note added: "Air Suspension"
- note added: "Aux Fuse and Switch Sensor"
- note added: "Inverter Fuse Sensor"
- note added: "Lights Fuse and Switch Sensor"
- note added: "Spare"
- note removed: "Air Suspension Switch and Fuse Sensor"
- note removed: "Inverter Fuse and Switch Sensor"
- note removed: "Lights & Aux Fuse and Switch Sensor"
- note removed: "Spare Fuse Sensor"
- moved on the sheet: D9, R47

Commit message: First attempt at PCB design
Parts:
- removed C27, C33: 100nF, symbol Device:C_Small
- removed D9: 4V7, Diode_THT:D_DO-41_SOD81_P10.16mm_Horizontal, symbol Diode:1N47xxA
- removed R51, R52, R54, R60, R61, R62, R63, R68, R69, R70, R71, R76, R77, R78: 680, symbol Device:R
- removed R56, R66: 1k2, symbol Device:R
- removed unit 2 of U23
- removed unit 1 of U23
- added C29, C38, C39: 100nF, symbol Device:C_Small
- added C33: 0.33uF, symbol Device:C_Polarized_Small_US
- added C34: 0.1uF, Capacitor_THT:CP_Radial_Tantal_D5.0mm_P5.00mm, symbol Device:C_Polarized_Small_US
- added D7: 1N914, Diode_THT:D_DO-35_SOD27_P7.62mm_Horizontal, symbol Diode:1N914
- added K6: Relay_SPDT, symbol Relay:Relay_SPDT
- added Q7: STP40NF30L, Package_TO_SOT_THT:TO-220F-3_Vertical, symbol camper_van:STP40NF03L
- added Q8: 2N2222, Package_TO_SOT_THT:TO-18-3, symbol Transistor_BJT:BC107
- added R43, R55: 1k2, symbol Device:R
- added R46: 2k2, symbol Device:R
- added U20, U22: CNY17-3, symbol Isolator:CNY17-3
- added U24: RS485-TTL, Package_SO:SOIC-8_3.9x4.9mm_P1.27mm, symbol Interface_UART:ISL3178E
- added U25: LM7805, Package_TO_SOT_THT:TO-220-3_Vertical, symbol Regulator_Linear:LM7805_TO220
- added unit 1 of U27
- added unit 2 of U27
- R47: value 10k -> 180
- R50: value 680 -> 150; footprint (none) -> Resistor_THT:R_Axial_DIN0207_L6.3mm_D2.5mm_P10.16mm_Horizontal
- R53: value 680 -> 1k2
- renumbered C24 to C28, C38 to C31, C25 to C32, C28 to C35, C26 to C36, C32 to C37, C34 to C40, C35 to C41, C36 to C42, C37 to C43, C29 to C44, C31 to C45, C39 to C46, C40 to C47, C41 to C48, R59 to R44, R75 to R45, R55 to R51, R57 to R52, R65 to R54, R67 to R56, R72 to R57, R73 to R58, R74 to R59, R58 to R60, R64 to R61, R79 to R62, R80 to R63, R81 to R64, U24 to U21, U21 to U23, U22 to U26, U23 to U27, U25 to U28
Connections:
- net Aux SW: now also R55.2
- net Aux SW Fuse: now also R53.2
- net Duoetto Power SW Fuse: now also K6.11
- net Fuse Aux: now also A3.15 (D12/CIPO), C38.1, U27.16; no longer A3.21 (A2)
- net Fuse Duoetto Pwr: now also A3.7 (D4); no longer A3.8 (D5), R53.1
- net Fuse Fridge: now also A3.11 (D8); no longer A3.14 (D11/COPI)
- net Fuse Lights: now also A3.13 (D10/CS); no longer A3.19 (A0)
- net Fuse Pump: now also A3.23 (SDA/A4); no longer A3.10 (D7)
- net Fuse Spare: now also A3.25 (A6); no longer A3.23 (SDA/A4)
- net Fuse_Air: now also A3.9 (D6); no longer A3.12 (D9), R50.1
- net GND: now also C33.2, C34.2, Q7.3 (S), R46.2, U20.2, U24.5 (GND), U25.2 (GND), U27.2, U27.3
- net GNDD: now also C29.2, C38.2, C39.2, Q8.1 (E), U22.2; no longer R50.2, R53.2
- net Solar: now also R43.2; no longer R47.2
- net Switch Aux: now also A3.16 (D13/SCK), C39.1, U27.13; no longer A3.22 (A3)
- net Switch Duoetto Pwr: now also A3.8 (D5); no longer A3.9 (D6)
- net Switch Fridge: now also A3.12 (D9); no longer A3.15 (D12/CIPO)
- net Switch Lights: now also A3.14 (D11/COPI); no longer A3.20 (A1)
- net Switch Pump: now also A3.24 (SCL/A5); no longer A3.11 (D8)
- net Switch Spare: now also A3.26 (A7); no longer A3.24 (SCL/A5)
- net Switch_Air: now also A3.10 (D7); no longer A3.13 (D10/CS)
- net VCC_3V3: now also D7.1 (K), K6.A1, U24.8 (VCC); no longer U21.10, U21.11, U21.14, U21.15, U26.10, U26.11, U26.14, U26.15, U27.10, U27.11, U28.10, U28.11, U28.14, U28.15
- net VCC_FS_9V5: now also C33.1, U25.1 (VI)
- net Tx: now reaches A3.1 (D1/TX)
- net Tx: now also U24.4 (DI)
- net Rx: now reaches A3.2 (D0/RX)
- net Rx: now also U24.1 (RO)
- net at R47.1: now also A3.22 (A3); no longer A3.25 (A6)
- net En: now reaches A3.5 (D2)
- net En: now also U24.2 (~{RE}), U24.3 (DE)
- net Fuse Duoetto 12V: no longer names the net of C30.1, U21.12
- net Fuse Duoetto 12V: now also A3.20 (A1); no longer A3.6 (D3)
- net Fuse Inverter: no longer names the net of C31.1, U21.9
- net Fuse Inverter: now also A3.21 (A2); no longer A3.7 (D4)
- new net: A3.19 (A0), C29.1, U20.4
- new net: R43.1, U20.1
- new net: R55.1, U27.4
- new net: R47.2, U22.1
- new net: Q7.1 (G), R46.1, U22.4
- new net: Q8.2 (B), R50.2
- new net: R53.1, U27.1
- new net: D7.2 (A), K6.A2, Q8.3 (C)
- new net +12V: U22.5
- new net Duoetto Pwr: K6.14
- new net Duoetto Pwr Ctrl: A3.6 (D3), R50.1
- new net Lights: Q7.2 (D)
- new net RS485 Rx: U24.6 (A)
- new net RS485 Tx: U24.7 (B)
- new net VCC_FS_3V3: C34.1, U20.5, U21.10, U21.11, U21.14, U21.15, U25.3 (VO), U26.10, U26.11, U26.14, U26.15, U27.10, U27.11, U27.14, U27.15, U28.10, U28.11, U28.14, U28.15
- no-connect marks 9 -> 7
Other:
- note added: "Solar Fuse Sensor"
- moved on the sheet: A3, C30, C31, C35, C36, C37, C40, C44, C45, R44, R45, R51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
