File: electrical/management_module.kicad_sch (KiCad schematic)
At the start: 88 parts, among them J1 Duoetto Remote, J2 Input Flow Sensor, J3 Output Flow Sensor, J4 Battery Box, J5 Starter Battery, J6 Fuse and Switch Box, J7 Fuse and Switch, J8 Lights, K2 G5Q-1, K3 G5Q-1, Q1 2N2222, Q2 D4184, Q3 2N2222, Q4 2N2222, Q5 D4184, SW1 SW_Push, U1 RS485-TTL, U2 LM7805, U3 MCP6004, U4 PC817, U5 DS18B20, U6 MCP6001U, U7 PC817

Commit message: Design has been split into 3x modules
- management module
- fuse and switch modules
- display module
Parts:
- removed A1: Arduino_Nano_ESP32, Module:Arduino_Nano, symbol MCU_Module:Arduino_Nano_ESP32
- removed D3, D8: 1N4001, Diode_THT:D_DO-41_SOD81_P10.16mm_Horizontal, symbol Diode:1N4001
- removed D5, D6: 1N914, Diode_THT:D_DO-35_SOD27_P7.62mm_Horizontal, symbol Diode:1N914
- removed J1: Duoetto Remote, Connector_Molex:Molex_Mini-Fit_Jr_5569-02A1_2x01_P4.20mm_Horizontal, symbol Connector:Conn_01x02_Pin
- removed J2: Input Flow Sensor, Connector_Molex:CONN_SD-172648-0000_02_MOL, symbol Connector:Conn_01x03_Pin
- removed J3: Output Flow Sensor, Connector_Molex:CONN_SD-172648-0000_02_MOL, symbol Connector:Conn_01x03_Pin
- removed J4: Battery Box, Connector_Molex:Molex_Mini-Fit_Jr_5569-16A2_2x08_P4.20mm_Horizontal, symbol Connector:Conn_01x16_Pin
- removed J5: Starter Battery, Connector_Molex:Molex_Mini-Fit_Jr_5569-02A2_2x01_P4.20mm_Horizontal, symbol Connector:Conn_01x01_Pin
- removed J6: Fuse and Switch Box, Connector_Molex:Molex_Mini-Fit_Jr_5569-06A1_2x03_P4.20mm_Horizontal, symbol Connector:Conn_01x06_Pin
- removed J7: Fuse and Switch, Connector_Molex:Molex_Mini-Fit_Jr_5569-02A1_2x01_P4.20mm_Horizontal, symbol Connector:Conn_01x02_Pin
- removed J8: Lights, Connector_Molex:Molex_Mini-Fit_Jr_5569-02A1_2x01_P4.20mm_Horizontal, symbol Connector:Conn_01x02_Pin
- removed K2, K3: G5Q-1, Relay_THT:Relay_SPDT_Omron-G5Q-1, symbol Relay:G5Q-1
- removed Q1: 2N2222, Package_TO_SOT_THT:TO-18-3, symbol Transistor_BJT:BC107
- removed Q2: D4184, symbol Simulation_SPICE:NMOS
- removed R2: 1k, symbol Device:R
- removed R32, R36: 5k9, symbol Device:R
- removed R39: 4k7, symbol Device:R
- removed R4: 10K 1%, Resistor_THT:R_Axial_DIN0207_L6.3mm_D2.5mm_P10.16mm_Horizontal, symbol Device:R
- removed U1: RS485-TTL, Package_SO:SOIC-8_3.9x4.9mm_P1.27mm, symbol Interface_UART:ISL3178E
- removed U2: LM7805, Package_TO_SOT_THT:TO-220-3_Vertical, symbol Regulator_Linear:LM7805_TO220
- removed U3: MCP6004, symbol Amplifier_Operational:MCP6004
- removed U5: DS18B20, Package_TO_SOT_THT:TO-92_Inline, symbol Sensor_Temperature:DS18B20
- removed U6: MCP6001U, symbol Amplifier_Operational:MCP6001U
- removed U7: PC817, Package_DIP:DIP-4_W7.62mm, symbol Isolator:PC817
- added A2: Arduino_Nano_ESP32, Module:Arduino_Nano, symbol MCU_Module:Arduino_Nano_ESP32
- added D2, D3: 1N914, Diode_THT:D_DO-35_SOD27_P7.62mm_Horizontal, symbol Diode:1N914
- added D5, D6: 1N4001, Diode_THT:D_DO-41_SOD81_P10.16mm_Horizontal, symbol Diode:1N4001
- added J10: Input Flow Sensor, Connector_Molex:CONN_SD-172648-0000_02_MOL, symbol Connector:Conn_01x03_Pin
- added J11: Output Flow Sensor, Connector_Molex:CONN_SD-172648-0000_02_MOL, symbol Connector:Conn_01x03_Pin
- added J12: Lights, Connector_Molex:Molex_Mini-Fit_Jr_5569-02A1_2x01_P4.20mm_Horizontal, symbol Connector:Conn_01x02_Pin
- added J13: Duoetto Remote, Connector_Molex:Molex_Mini-Fit_Jr_5569-02A1_2x01_P4.20mm_Horizontal, symbol Connector:Conn_01x02_Pin
- added J14: Fuse and Switch, Connector_Molex:Molex_Mini-Fit_Jr_5569-02A1_2x01_P4.20mm_Horizontal, symbol Connector:Conn_01x02_Pin
- added J15: Fuse and Switch Box, Connector_Molex:Molex_Mini-Fit_Jr_5569-06A1_2x03_P4.20mm_Horizontal, symbol Connector:Conn_01x06_Pin
- added J16: Battery Box, Connector_Molex:Molex_Mini-Fit_Jr_5569-16A2_2x08_P4.20mm_Horizontal, symbol Connector:Conn_01x16_Pin
- added J17: Starter Battery, Connector_Molex:Molex_Mini-Fit_Jr_5569-02A2_2x01_P4.20mm_Horizontal, symbol Connector:Conn_01x01_Pin
- added K5, K6: G5Q-1, Relay_THT:Relay_SPDT_Omron-G5Q-1, symbol Relay:G5Q-1
- added Q1: D4184, symbol Simulation_SPICE:NMOS
- added Q5: 2N2222, Package_TO_SOT_THT:TO-18-3, symbol Transistor_BJT:BC107
- added R14: 10k, symbol Device:R
- added R15: 5k9, symbol Device:R
- added R40, R42: 35.7K 1%, Resistor_THT:R_Axial_DIN0207_L6.3mm_D2.5mm_P10.16mm_Horizontal, symbol Device:R
- added R41: 10K 1%, Resistor_THT:R_Axial_DIN0207_L6.3mm_D2.5mm_P10.16mm_Horizontal, symbol Device:R
- added U10: MCP6001U, symbol Amplifier_Operational:MCP6001U
- added U5: PC817, Package_DIP:DIP-4_W7.62mm, symbol Isolator:PC817
- added U6: LM7805, Package_TO_SOT_THT:TO-220-3_Vertical, symbol Regulator_Linear:LM7805_TO220
- added U7: RS485-TTL, Package_SO:SOIC-8_3.9x4.9mm_P1.27mm, symbol Interface_UART:ISL3178E
- added U8: DS18B20, Package_TO_SOT_THT:TO-92_Inline, symbol Sensor_Temperature:DS18B20
- added U9: MCP6004, symbol Amplifier_Operational:MCP6004
- R1: value 150 -> 4k7; footprint Resistor_THT:R_Axial_DIN0207_L6.3mm_D2.5mm_P10.16mm_Horizontal -> (none)
- R10: value 10K 1% -> 1k; footprint Resistor_THT:R_Axial_DIN0207_L6.3mm_D2.5mm_P10.16mm_Horizontal -> (none)
- R11, R17: value 35.7K 1% -> 150
- R12: value 10K 1% -> 150
- R13: value 150 -> 5k9; footprint Resistor_THT:R_Axial_DIN0207_L6.3mm_D2.5mm_P10.16mm_Horizontal -> (none)
- R16: value 150 -> 10k; footprint Resistor_THT:R_Axial_DIN0207_L6.3mm_D2.5mm_P10.16mm_Horizontal -> (none)
- R18: value 10K 1% -> 154k; footprint Resistor_THT:R_Axial_DIN0207_L6.3mm_D2.5mm_P10.16mm_Horizontal -> (none)
- R19: value 4k7 -> 154k
- R20: value 100 -> 35.7K 1%; footprint (none) -> Resistor_THT:R_Axial_DIN0207_L6.3mm_D2.5mm_P10.16mm_Horizontal
- R21: value 4k7 -> 10K 1%; footprint (none) -> Resistor_THT:R_Axial_DIN0207_L6.3mm_D2.5mm_P10.16mm_Horizontal
- R22: value 5k9 -> 154k
- R23, R37: value 10k -> 154k
- R24, R26: value 154k -> 35.7K 1%; footprint (none) -> Resistor_THT:R_Axial_DIN0207_L6.3mm_D2.5mm_P10.16mm_Horizontal
- R25, R27: value 154k -> 10K 1%; footprint (none) -> Resistor_THT:R_Axial_DIN0207_L6.3mm_D2.5mm_P10.16mm_Horizontal
- R3: value 35.7K 1% -> 100; footprint Resistor_THT:R_Axial_DIN0207_L6.3mm_D2.5mm_P10.16mm_Horizontal -> (none)
- R30: value 154k -> 5k9
- R31: value 154k -> 10k
- R38: value 1k -> 154k
- R43: value 10k -> 10K 1%; footprint (none) -> Resistor_THT:R_Axial_DIN0207_L6.3mm_D2.5mm_P10.16mm_Horizontal
- R7: value 35.7K 1% -> 4k7; footprint Resistor_THT:R_Axial_DIN0207_L6.3mm_D2.5mm_P10.16mm_Horizontal -> (none)
- R8: value 10K 1% -> 4k7; footprint Resistor_THT:R_Axial_DIN0207_L6.3mm_D2.5mm_P10.16mm_Horizontal -> (none)
- R9: value 35.7K 1% -> 1k; footprint Resistor_THT:R_Axial_DIN0207_L6.3mm_D2.5mm_P10.16mm_Horizontal -> (none)
- renumbered C4 to C10, C3 to C11, C9 to C3, C10 to C4, C7 to C5, C8 to C6, C11 to C7, C5 to C8, C6 to C9, Q5 to Q2, R41 to R2, R42 to R32, R44 to R36, R45 to R39, R40 to R4, R46 to R44, R47 to R45
Connections:
- net +12V: now also R7.1, R8.1, D2.1 (K), D3.1 (K), J16.15 (Pin_15), K5.1, K5.2, K6.1; no longer R21.1
- net +5V: now also J10.1 (Pin_1), J11.1 (Pin_1), J16.5 (Pin_5), U10.5 (V+), U6.3 (VO), U7.8 (VCC), U8.3 (V_{DD}), U9.4 (V+)
- net 12V Power On/Off: now also R12.2, A2.16 (D13/SCK); no longer R13.2
- net Battery 1 In Sensor: now also R24.1, J16.9 (Pin_9); no longer R5.1
- net Battery 1 Out Sensor: now also J16.11 (Pin_11), R40.1; no longer R9.1
- net Battery 2: now also R20.1, D3.2 (A), J15.3 (Pin_3), K6.5, Q5.3 (C); no longer D7.2 (A)
- net Battery 2 In Sensor: now also R26.1, J16.10 (Pin_10); no longer R7.1
- net Battery 2 On/Off: now also R17.1, A2.13 (D10/CS); no longer R16.1
- net Battery 2 On/Off Switch Sensor: now also R20.2, R21.1, A2.12 (D9); no longer R17.2, R18.1
- net Battery 2 Out Sensor: now also J16.12 (Pin_12), R42.1; no longer R11.1
- net Battery Box Fan: now also J16.3 (Pin_3), Q1.1 (D)
- net GND: now also D4.1 (K), R1.2, R16.2, R21.2, R25.2, R27.2, R31.2, A2.29 (GND), A2.4 (GND), D5.1 (K), J10.3 (Pin_3), J11.3 (Pin_3), J12.2 (Pin_2), J15.4 (Pin_4), J15.6 (Pin_6), J16.16 (Pin_16), Q1.3 (S), Q5.1 (E), R14.2, R41.2, U10.2 (V-), U5.2, U6.2 (GND), U7.5 (GND), U8.1 (GND), U9.11 (V-); no longer D7.1 (K), R10.2, R12.2, R18.2, R19.2, R23.2, R37.2, R8.2
- net Input Flow Sensor: now also A2.10 (D7), J10.2 (Pin_2)
- net Light Control: now also R10.1, A2.9 (D6); no longer R38.1
- net Output Flow Sensor: now also A2.11 (D8), J11.2 (Pin_2)
- net RS485 Rx: now also J13.2 (Pin_2), J14.1 (Pin_1), J16.1 (Pin_1), U7.6 (A)
- net RS485 Tx: now also J13.1 (Pin_1), J14.2 (Pin_2), J16.2 (Pin_2), U7.7 (B)
- net Solar Switch: now also Q3.3 (C), R5.1; no longer R3.1
- net VIN: now also D7.1 (K), A2.30 (VIN), D6.1 (K), U6.1 (VI); no longer D4.1 (K)
- net at R24.2, R25.1: now also R22.1; no longer C10.1
- net at C10.2: now also R30.1, A2.22 (A3), U9.14; no longer R22.1
- net at R3.2: now also R1.1, Q1.2 (G)
- net at R4.1: now also U5.3; no longer U4.3
- net at C12.1, R36.2: now also U10.1 (+)
- net at R38.2: now also C10.1, R35.1; no longer U4.1
- net at U4.4: now also R7.2
- net at R33.1: now also R32.2, U10.3 (-)
- net at R28.2, R29.1: now also U9.9 (-)
- net at Q4.2 (B): now also R12.1; no longer R16.2
- net at Q4.3 (C): now also D2.2 (A), K5.5; no longer R17.1
- net at C9.1: now also R34.2, U9.10 (+); no longer R27.2
- net Battery 2 Relay: now reaches D4.2 (A)
- net Battery 2 Relay: now also J16.14 (Pin_14), K6.3
- net at R23.1: now also R26.2, R27.1; no longer R22.2
- net at R19.1: now also C5.1, R23.2; no longer R20.2
- net at C8.2, R28.1: now also A2.21 (A2), U9.8
- net at C4.1: now also R18.2, U9.3 (+); no longer R35.2
- net at R43.1: now also R38.1, R42.2; no longer R32.2
- net at R13.1: now also C3.2, A2.19 (A0), U9.1; no longer Q3.2 (B)
- net at R30.2, R31.1: now also U9.13 (-); no longer C5.1
- net at C5.2: now also A2.20 (A1), R15.1, U9.7
- net at C7.2, R32.1: now also A2.23 (SDA/A4), U10.4
- net at R5.2, R6.1: now also A2.7 (D4); no longer R34.1
- net at SW1.1: now also A2.3 (~{RESET})
- net at R44.1: now also J17.1 (Pin_1)
- net at Q2.1 (D): now also J12.1 (Pin_1)
- net at C6.1: now also R19.2, U9.5 (+); no longer R31.2
- net at R37.1: now also R40.2, R41.1
- net at C11.1: now also R35.2, U9.12 (+); no longer R25.2
- new net: A2.1 (D1/TX), U7.4 (DI)
- new net: A2.2 (D0/RX), U7.1 (RO)
- new net: A2.5 (D2), U7.2 (~{RE}), U7.3 (DE)
- new net: A2.6 (D3), R11.2
- new net: A2.8 (D5), R9.1
- new net: Q3.2 (B), R11.1
- new net: R3.1, U4.3
- new net: C8.1, R34.1, R37.2
- new net: C3.1, R18.1, R22.2
- new net: R13.2, R14.1, U9.2 (-)
- new net: Q5.2 (B), R17.2
- new net: R15.2, R16.1, U9.6 (-)
- new net: R10.2, U5.1
- new net: R8.2, U5.4
- new net: R9.2, U4.1
- new net Battery 1 Relay: D5.2 (A), J16.13 (Pin_13), K6.4
- new net Battery 1 Vin: D6.2 (A), J16.7 (Pin_7)
- new net Battery 2 Vin: D7.2 (A), J16.8 (Pin_8)
- new net Power On/Off A: J15.1 (Pin_1), K6.2
- new net Power On/Off B: J15.2 (Pin_2), K5.3
- new net Solar Charge Battery 2: J15.5 (Pin_5), J16.6 (Pin_6)
- new net Temperature Sensors: A2.26 (A7), J16.4 (Pin_4), U8.2 (DQ)
Other:
- note removed: "Battery 2 On/Off"
- note removed: "Solar/50A charge Battery 2"
- moved on the sheet: C10, C11, C12, C3, C4, C5, C6, C7, C8, C9, Q2, R2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

Commit message: lots of redesign
Parts:
- removed C1: 0.33uF, Capacitor_THT:CP_Radial_Tantal_D5.0mm_P5.00mm, symbol Device:C_Polarized_Small_US
- removed C10, C11, C7, C8, C9: 1uF, symbol Device:C
- removed D2: 1N914, Diode_THT:D_DO-35_SOD27_P7.62mm_Horizontal, symbol Diode:1N914
- removed J17: Starter Battery, Connector_Molex:Molex_Mini-Fit_Jr_5569-02A2_2x01_P4.20mm_Horizontal, symbol Connector:Conn_01x01_Pin
- removed K5: G5Q-1, Relay_THT:Relay_SPDT_Omron-G5Q-1, symbol Relay:G5Q-1
- removed Q1, Q2: D4184, symbol Simulation_SPICE:NMOS
- removed Q3, Q4: 2N2222, Package_TO_SOT_THT:TO-18-3, symbol Transistor_BJT:BC107
- removed R21, R25: 10K 1%, Resistor_THT:R_Axial_DIN0207_L6.3mm_D2.5mm_P10.16mm_Horizontal, symbol Device:R
- removed R24: 35.7K 1%, Resistor_THT:R_Axial_DIN0207_L6.3mm_D2.5mm_P10.16mm_Horizontal, symbol Device:R
- removed R28: 5k9, symbol Device:R
- removed R29, R33: 10k, symbol Device:R
- removed R3, R4: 100, symbol Device:R
- removed R34: 154k, symbol Device:R
- removed R7, R8: 4k7, symbol Device:R
- removed U10: MCP6001U, symbol Amplifier_Operational:MCP6001U
- removed U4, U5: PC817, Package_DIP:DIP-4_W7.62mm, symbol Isolator:PC817
- removed U9: MCP6004, symbol Amplifier_Operational:MCP6004
- added C1, C16, C19, C2, C21, C3, C4, C5: 100nF, symbol Device:C_Small
- added C13, C15, C18, C20: 1uF, symbol Device:C
- added C17: 22uF, symbol Device:C_Polarized_Small_US
- added C6, C7: 0.33uF, symbol Device:C_Polarized_Small_US
- added D2, D3: 1N4001, Diode_THT:D_DO-41_SOD81_P10.16mm_Horizontal, symbol Diode:1N4001
- added J16: Starter Battery, Connector_Molex:Molex_Mini-Fit_Jr_5569-02A2_2x01_P4.20mm_Horizontal, symbol Connector:Conn_01x01_Pin
- added Q1, Q2, Q3, Q4, Q5, Q6: STP40NF30L, Package_TO_SOT_THT:TO-220F-3_Vertical, symbol Transistor_FET:STP40NF03L
- added R1, R10, R17, R2: 4k7, symbol Device:R
- added R13, R19, R9: ??, symbol Device:R
- added R14, R15, R18: 390, symbol Device:R
- added R16: 82R 2W, symbol Device:R
- added R46: 10k, symbol Device:R
- added U10, U11, U4, U5, U6, U7, U8, U9: CNY17-3, symbol Isolator:CNY17-3
- added U13, U21: MCP6004, symbol Amplifier_Operational:MCP6004
- added U14: MCP6002-xP, symbol Amplifier_Operational:MCP6002-xP
- added U16: BA00, Package_TO_SOT_THT:TO-220-5_P3.4x3.8mm_StaggerOdd_Lead7.13mm_TabDown, symbol camper_van:BA00
- added U18, U19, U20: IL300, symbol Isolator_Analog:IL300
- K5: renamed from K6; value G5Q-1 -> G5V-1
- R11: value 150 -> 180; footprint Resistor_THT:R_Axial_DIN0207_L6.3mm_D2.5mm_P10.16mm_Horizontal -> (none)
- R12: value 150 -> 390; footprint Resistor_THT:R_Axial_DIN0207_L6.3mm_D2.5mm_P10.16mm_Horizontal -> (none)
- R20: value 35.7K 1% -> ??; footprint Resistor_THT:R_Axial_DIN0207_L6.3mm_D2.5mm_P10.16mm_Horizontal -> (none)
- R26: value 35.7K 1% -> 5k9; footprint Resistor_THT:R_Axial_DIN0207_L6.3mm_D2.5mm_P10.16mm_Horizontal -> (none)
- R27, R45: value 10K 1% -> 10k; footprint Resistor_THT:R_Axial_DIN0207_L6.3mm_D2.5mm_P10.16mm_Horizontal -> (none)
- R30: value 5k9 -> 154k
- R31: value 10k -> 68k
- R32: value 5k9 -> 10k
- R36, R37, R38: value 154k -> 22k
- R39: value 154k -> 1k2
- R40: value 35.7K 1% -> 1k2; footprint Resistor_THT:R_Axial_DIN0207_L6.3mm_D2.5mm_P10.16mm_Horizontal -> (none)
- R41: value 10K 1% -> 1k2; footprint Resistor_THT:R_Axial_DIN0207_L6.3mm_D2.5mm_P10.16mm_Horizontal -> (none)
- R42, R44: value 35.7K 1% -> 100k; footprint Resistor_THT:R_Axial_DIN0207_L6.3mm_D2.5mm_P10.16mm_Horizontal -> (none)
- R43: value 10K 1% -> 100k; footprint Resistor_THT:R_Axial_DIN0207_L6.3mm_D2.5mm_P10.16mm_Horizontal -> (none)
- R5: value 35.7K 1% -> 4k7; footprint Resistor_THT:R_Axial_DIN0207_L6.3mm_D2.5mm_P10.16mm_Horizontal -> (none)
- R6: value 10K 1% -> 180; footprint Resistor_THT:R_Axial_DIN0207_L6.3mm_D2.5mm_P10.16mm_Horizontal -> (none)
- R7: renamed from R9; value 1k -> 180
- R8: renamed from R10; value 1k -> 180
- renumbered C5 to C10, C6 to C11, C2 to C14, C3 to C8, C4 to C9, D3 to D4, D4 to D5, D5 to D6, D6 to D7, D7 to D8, J15 to J13, J13 to J14, J14 to J15, J16 to J17, Q5 to Q7, R17 to R21, R13 to R22, R14 to R23, R15 to R24, R16 to R25, R18 to R28, R19 to R29, R1 to R3, R22 to R33, R23 to R34, R2 to R4, U8 to U12, U6 to U15, U7 to U17
Connections:
- net +12V: now also D1.2 (A), D2.2 (A), U18.2, U19.2, U20.2, U5.5, U6.5, U7.5; no longer D1.1 (K), D4.1 (K), K5.1
- net Battery 1 Out Sensor: now also R19.2; no longer R40.1
- net Battery 1 Vin: now also R42.1
- net Battery 2: now also R9.2; no longer D4.2 (A), K5.5, Q7.3 (C), R20.1
- net Battery 2 On/Off: now also A2.10 (D7); no longer A2.13 (D10/CS)
- net Battery 2 On/Off Switch Sensor: now also A2.9 (D6), R12.1, U8.4; no longer A2.12 (D9), R20.2
- net Battery 2 Out Sensor: now also R20.2; no longer R42.1
- net Battery 2 Vin: now also R43.1
- net Battery Box Fan: now also D1.1 (K), Q2.2 (D)
- net GND: now also R32.2, R5.2, C17.2, C20.2, C21.2, C6.2, C7.2, Q1.3 (S), Q2.3 (S), Q3.3 (S), Q4.3 (S), R2.2, R46.2, U10.2, U11.2, U16.1 (CTL), U16.3 (GND), U18.4, U19.4, U20.4, U21.11 (V-), U21.2 (-), U21.6 (-), U21.9 (-), U8.2, U9.2; no longer A2.29 (GND), A2.4 (GND), C11.2, C12.2, C9.2, Q7.1 (E), R23.2, R25.2, R27.2, R31.2, R41.2, R43.2, R45.2, R6.2, SW1.2
- net Input Flow Sensor: now also A2.15 (D12/CIPO); no longer A2.10 (D7)
- net Output Flow Sensor: now also A2.16 (D13/SCK); no longer A2.11 (D8)
- net Power On/Off B: now also Q5.2 (D)
- net RS485 Rx: now also J17.2 (Pin_2); no longer J17.1 (Pin_1)
- net RS485 Tx: now also J17.1 (Pin_1); no longer J17.2 (Pin_2)
- net Solar Charge Battery 2: now also D3.1 (K), Q4.2 (D), R1.1; no longer J13.5 (Pin_5)
- net VIN: now also J13.1 (Pin_1), C7.1, D3.2 (A), R10.1, R16.1, R17.1, U16.2 (VIN), U4.5; no longer A2.30 (VIN), U15.1 (VI)
- net at R35.1, R38.2: now also U14.7
- net at R30.1: now also C12.1, R35.2; no longer A2.22 (A3)
- net Tx: now reaches A2.1 (D1/TX), U17.4 (DI)
- net at A2.14 (D11/COPI): now also R8.1
- net at A2.19 (A0), C8.2, R22.1: now also C4.1, U13.1
- net Rx: now reaches A2.2 (D0/RX), U17.1 (RO)
- net at A2.20 (A1), C10.2, R24.1: now also C5.1, U13.8
- net at A2.21 (A2): now also C12.2, R26.1, C3.1, U14.1
- net at R32.1: now also R31.2, U16.5 (ADJ); no longer A2.23 (SDA/A4)
- net En: now reaches A2.5 (D2), U17.2 (~{RE}), U17.3 (DE)
- net at R11.2: now also U7.1; no longer A2.6 (D3)
- net at R7.1: now also A2.13 (D10/CS); no longer A2.8 (D5)
- net at R26.2, R27.1: now also U14.2 (-); no longer R34.1
- net at R4.1: now also Q3.1 (G), U6.4
- net Solar Charge Battery 2 On: now reaches R11.1
- net Solar Charge Battery 2 On: now also A2.7 (D4)
- net at R36.2: now also R33.1, U13.7; no longer C12.1
- net at R3.1: now also Q2.1 (G), U5.4
- net at R37.2: now also R34.1, U13.14
- net at R22.2, R23.1: now also U13.2 (-)
- net at C9.1, R28.2: now also U13.3 (+)
- net at R24.2, R25.1: now also U13.9 (-)
- net at R44.1: now also J16.1 (Pin_1)
- net at R8.2: now also U6.1
- net at J12.1 (Pin_1): now also D2.1 (K), Q3.2 (D)
- net at R30.2: now also C13.1, U14.3 (+); no longer R31.1
- net at R39.2: now also U18.1; no longer R36.1
- net at R7.2: now also U5.1
- net at C11.1, R29.2: now also U13.10 (+)
- net +5V renamed VCC_3V3
- net VCC_3V3: now also D4.1 (K), K5.1, Q7.3 (C), R45.1, C15.1, C16.1, C18.1, C19.1, C20.1, C21.1, U10.5, U11.5, U13.4 (V+), U14.8 (V+), U21.4 (V+), U8.5, U9.5
- net 12V Power On/Off renamed GNDD
- net GNDD: now also A2.29 (GND), A2.4 (GND), Q7.1 (E), SW1.2, C1.2, C2.2, C3.2, C4.2, C5.2, R14.2, R15.2, R18.2, U4.2, U5.2, U6.2, U7.2; no longer A2.16 (D13/SCK)
- net Battery 1 In Sensor: no longer names the net of J17.9 (Pin_9)
- net Battery 2 In Sensor: no longer names the net of J17.10 (Pin_10)
- net Battery 2 In Sensor: no longer R26.1
- removed net Light Control: A2.9 (D6), R8.1
- net Power On/Off A: no longer names the net of K5.2
- net Power On/Off A: now also Q5.3 (S), Q6.3 (S); no longer J13.1 (Pin_1)
- net Solar Switch: no longer names the net of R5.1
- net Solar Switch: now also Q4.1 (G), U7.4; no longer D1.2 (A)
- new net: R44.2, U20.3, U21.10 (+)
- new net: R41.1, U21.8
- new net: R20.1, U11.1
- new net: R43.2, U19.3, U21.5 (+)
- new net: R19.1, U10.1
- new net: Q1.1 (G), R2.1, U4.4
- new net: R40.1, U21.7
- new net: R9.1, U8.1
- new net: R39.1, U21.1
- new net: R41.2, U20.1
- new net: R38.1, U14.5 (+), U20.6
- new net: R36.1, U13.5 (+), U18.6
- new net: R40.2, U19.1
- new net: D4.2 (A), K5.5
- new net: Q6.2 (D), R16.2
- new net: R42.2, U18.3, U21.3 (+)
- new net: R13.1, U9.1
- new net: R37.1, U13.12 (+), U19.6
- new net: J13.5 (Pin_5), R13.2
- new net: R45.2, R46.1, U21.12 (+)
- new net: R6.2, U4.1
- new net: Q1.2 (D), R1.2
- new net: U21.13 (-), U21.14
- new net Batteries Off: A2.12 (D9), Q6.1 (G), R17.2
- new net Batteries On: A2.11 (D8), Q5.1 (G), R10.2
- new net Battery 1 Out Digital: A2.22 (A3), C2.1, R14.1, U10.4
- new net Battery 2 Out Digital: A2.23 (SDA/A4), C1.1, R15.1, U11.4
- new net GNDA: C11.2, C13.2, C15.2, C16.2, C18.2, C19.2, C9.2, R23.2, R25.2, R27.2, U13.11 (V-), U13.13 (-), U13.6 (-), U14.4 (V-), U14.6 (-), U18.5, U19.5, U20.5
- new net Solar Charge Battery 2 Off: A2.8 (D5), R6.1
- new net Solar Charge Battery 2 Switch Sensor: A2.6 (D3), R18.1, U9.4
- new net VCC_MM_9V5: A2.30 (VIN), C17.1, C6.1, R31.1, U15.1 (VI), U16.4 (VOUT)
- no-connect marks 9 -> 16
Other:
- note added: "Solar Charge Battery 2 Switch"
- note removed: "12V Power On/Off"
- moved on the sheet: C10, C11, C14, C8, C9, D4, D5, D6, J10, J11, J12, J13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

Commit message: work in progress
Parts:
- removed Q5, Q6: STP40NF30L, Package_TO_SOT_THT:TO-220F-3_Vertical, symbol Transistor_FET:STP40NF03L
- removed R10: 4k7, symbol Device:R
- removed R16: 82R 2W, symbol Device:R
- removed R6: 180, symbol Device:R
- removed U4: CNY17-3, symbol Isolator:CNY17-3
- added C1, C2: 100nF, symbol Device:C_Small
- added Q5, Q6: STP40NF30L, Package_TO_SOT_THT:TO-220F-3_Vertical, symbol camper_van:STP40NF03L
- added Q8: 2N2222, Package_TO_SOT_THT:TO-18-3, symbol Transistor_BJT:BC107
- added R105: 150, Resistor_THT:R_Axial_DIN0207_L6.3mm_D2.5mm_P10.16mm_Horizontal, symbol Device:R
- added R13, R14: 4k7, symbol Device:R
- J13: value Fuse and Switch Box -> Conn_01x06_Pin; footprint Connector_Molex:Molex_Mini-Fit_Jr_5569-06A1_2x03_P4.20mm_Horizontal -> (none)
- Q1: renamed from Q4; symbol Transistor_FET:STP40NF03L -> camper_van:STP40NF03L
- Q2, Q3: symbol Transistor_FET:STP40NF03L -> camper_van:STP40NF03L
- Q4: renamed from Q1; symbol Transistor_FET:STP40NF03L -> camper_van:STP40NF03L
- R1: value 4k7 -> 100 2W
- R17: value 4k7 -> 41R 2W
- R2: renamed from R5; value 4k7 -> 1M
- renumbered C8 to C10, C9 to C11, C10 to C12, C11 to C13, C12 to C14, C13 to C15, C14 to C16, C15 to C17, C16 to C18, C17 to C19, C18 to C20, C19 to C21, C20 to C22, C21 to C23, C1 to C3, C2 to C4, C3 to C5, C4 to C6, C5 to C7, C6 to C8, C7 to C9, D3 to D1, D1 to D2, D2 to D3, R11 to R10, R12 to R11, R18 to R12, R14 to R15, R15 to R16, R19 to R18, R20 to R19, R21 to R20, R22 to R21, R23 to R22, R24 to R23, R25 to R24, R26 to R25, R27 to R26, R28 to R27, R29 to R28, R30 to R29, R31 to R30, R32 to R31, R33 to R32, R34 to R33, R35 to R34, R36 to R35, R37 to R36, R38 to R37, R39 to R38, R40 to R39, R41 to R40, R42 to R41, R43 to R42, R44 to R43, R45 to R44, R46 to R45, R2 to R5, R9 to R6, R13 to R7, R7 to R8, R8 to R9, U11 to U10, U12 to U11, U13 to U12, U14 to U13, U15 to U14, U16 to U15, U17 to U16, U18 to U17, U19 to U18, U20 to U19, U21 to U20, U5 to U4, U6 to U5, U7 to U6, U8 to U7, U9 to U8, U10 to U9
Connections:
- net Power On/Off B is gone; now on net +12V: J13.2 (Pin_2)
- net Solar Charge Battery 2 Off is gone; now on net Battery 2 On/Off Switch Sensor: A2.8 (D5)
- net Batteries On: now also A2.10 (D7), C2.2, Q6.1 (G), R14.1; no longer A2.11 (D8)
- net Battery 1 Relay: now also D6.1 (K); no longer D6.2 (A)
- net Battery 2 On/Off: now also A2.9 (D6); no longer A2.10 (D7)
- net Battery 2 On/Off Switch Sensor: now also R105.1; no longer A2.9 (D6)
- net Battery 2 Relay: now also D5.1 (K); no longer D5.2 (A)
- net GND: now also Q6.3 (S), R13.2, R14.2; no longer D5.1 (K), D6.1 (K), J13.4 (Pin_4)
- net GNDD: now also Q8.1 (E)
- net Solar Charge Battery 2: now also R1.2; no longer R1.1
- net VCC_3V3: now also Q8.3 (C)
- net VIN: now also D5.2 (A), D6.2 (A), J13.4 (Pin_4), J17.10 (Pin_10), J17.9 (Pin_9); no longer J13.1 (Pin_1), R17.1
- net at R8.1: now also A2.11 (D8); no longer A2.13 (D10/CS)
- net at R9.1: now also A2.12 (D9); no longer A2.14 (D11/COPI)
- net at Q1.1 (G), R2.1: now also C1.1; no longer U6.4
- net Solar Charge Battery 2 SW: now reaches Q4.1 (G), R5.1
- net Solar Charge Battery 2 SW: now also J13.5 (Pin_5), R7.2, U6.4, C1.2
- net at K5.2: now also R17.2, Q5.2 (D)
- net at Q4.2 (D): now also R1.1; no longer R1.2
- removed net Batteries Off: A2.12 (D9), R17.2
- net Battery 1 Out Digital renamed Battery 1 Fuse Digital
- net Battery 1 Out Sensor renamed Battery 1 Fuse Sensor
- net Battery 2 renamed Battery 2 SW
- net Battery 2 Out Digital renamed Battery 2 Fuse Digital
- net Battery 2 Out Sensor renamed Battery 2 Fuse Sensor
- new net: Q6.2 (D), R17.1
- new net: Q8.2 (B), R105.2
- new net: C2.1, Q5.1 (G), R13.1
- new net Power On/Off SW: J13.1 (Pin_1), Q5.3 (S)
- no-connect marks 16 -> 15
Other:
- note removed: "Solar Charge Battery 2 Switch"
- moved on the sheet: D1, D5, D6, Q1, Q4, Q7, R1, R10, R11, R12, R2, R20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

Commit message: UPdated
Parts:
- removed J13: Conn_01x06_Pin, symbol Connector:Conn_01x06_Pin
- added J35: Power On/Off SW, symbol Connector:Conn_01x02_Socket
- added J36: Battewry 2, symbol Connector:Conn_01x04_Socket
- J32: renamed from J10; footprint Connector_Molex:CONN_SD-172648-0000_02_MOL -> (none)
- J33: renamed from J11; footprint Connector_Molex:CONN_SD-172648-0000_02_MOL -> (none)
- R11, R12: value 390 -> 680
- R16: renamed from R15; value 390 -> 680
- R17: renamed from R16; value 390 -> 680
- R19: renamed from R18; value ?? -> 1k2
- R20: renamed from R19; value ?? -> 1k2
- R3, R4, R5: value 4k7 -> 2k2
- SW14: renamed from SW1; footprint Button_Switch_SMD:SW_SPST_EVQP2 -> (none)
- renumbered J12 to J34, J14 to J37, J15 to J38, J16 to J39, J17 to J40, Q8 to Q7, Q7 to Q8, R105 to R15, R17 to R18, R20 to R21, R21 to R22, R22 to R23, R23 to R24, R24 to R25, R25 to R26, R26 to R27, R27 to R28, R28 to R29, R29 to R30, R30 to R31, R31 to R32, R32 to R33, R33 to R34, R34 to R35, R35 to R36, R36 to R37, R37 to R38, R38 to R39, R39 to R40, R40 to R41, R41 to R42, R42 to R43, R43 to R44, R44 to R45, R45 to R46
Connections:
- net +12V: now also J35.2 (Pin_2)
- net Battery 2 SW: now also J36.1 (Pin_1)
- net GND: now also J36.4 (Pin_4)
- net Power On/Off SW: now also J35.1 (Pin_1)
- net Solar Charge Battery 2 SW: now also J36.3 (Pin_3)
- net VIN: now also J36.2 (Pin_2)

Commit message: First attempt at PCB design
Parts:
- removed D2, D3: 1N4001, Diode_THT:D_DO-41_SOD81_P10.16mm_Horizontal, symbol Diode:1N4001
- removed J32: Input Flow Sensor, symbol Connector:Conn_01x03_Pin
- removed J33: Output Flow Sensor, symbol Connector:Conn_01x03_Pin
- removed J34: Lights, Connector_Molex:Molex_Mini-Fit_Jr_5569-02A1_2x01_P4.20mm_Horizontal, symbol Connector:Conn_01x02_Pin
- removed J35: Power On/Off SW, symbol Connector:Conn_01x02_Socket
- removed J36: Battewry 2, symbol Connector:Conn_01x04_Socket
- removed J37: Duoetto Remote, Connector_Molex:Molex_Mini-Fit_Jr_5569-02A1_2x01_P4.20mm_Horizontal, symbol Connector:Conn_01x02_Pin
- removed J38: Fuse and Switch, Connector_Molex:Molex_Mini-Fit_Jr_5569-02A1_2x01_P4.20mm_Horizontal, symbol Connector:Conn_01x02_Pin
- removed J40: Battery Box, Connector_Molex:Molex_Mini-Fit_Jr_5569-16A2_2x08_P4.20mm_Horizontal, symbol Connector:Conn_01x16_Pin
- removed Q2, Q3: STP40NF30L, Package_TO_SOT_THT:TO-220F-3_Vertical, symbol camper_van:STP40NF03L
- removed R11, R12, R16, R17: 680, symbol Device:R
- removed U4, U5: CNY17-3, symbol Isolator:CNY17-3
- added C2, C3, C4, C5: 100nF, symbol Device:C_Small
- added U4: ILQ615-3, symbol camper_van:ILQ615-3
- R15: renamed from R19; value 1k2 -> 680
- R16: renamed from R20; value 1k2 -> 680
- R3, R4: value 2k2 -> 47k
- R5: renamed from R6; value ?? -> 680
- R7: value ?? -> 680
- renumbered C6 to C10, C7 to C11, C8 to C12, C9 to C13, C10 to C14, C11 to C15, C12 to C16, C13 to C17, C14 to C18, C15 to C19, C16 to C20, C17 to C21, C18 to C22, C19 to C23, C20 to C24, C21 to C25, C22 to C26, C23 to C27, C2 to C6, C4 to C7, C3 to C8, C5 to C9, D4 to D2, D5 to D3, D6 to D4, D7 to D5, D8 to D6, J39 to J35, Q4 to Q2, Q5 to Q3, Q6 to Q4, Q7 to Q5, Q8 to Q6, R13 to R11, R14 to R12, R15 to R13, R18 to R14, R21 to R17, R22 to R18, R23 to R19, R24 to R20, R25 to R21, R26 to R22, R27 to R23, R28 to R24, R29 to R25, R30 to R26, R31 to R27, R32 to R28, R33 to R29, R34 to R30, R35 to R31, R36 to R32, R37 to R33, R38 to R34, R39 to R35, R40 to R36, R41 to R37, R42 to R38, R43 to R39, R44 to R40, R45 to R41, R46 to R42, R5 to R6, U11 to U10, U12 to U11, U13 to U12, U14 to U13, U15 to U14, U17 to U15, U18 to U16, U16 to U17, U19 to U18, U20 to U19, U7 to U5, U8 to U7, U9 to U8, U10 to U9
Connections:
- net +12V: now also R3.1, R4.1
- net Battery 1 Relay: now also D4.2 (A); no longer D4.1 (K)
- net Battery 2 On/Off Switch Sensor: now also C2.1
- net Battery 2 Relay: now also D3.2 (A); no longer D3.1 (K)
- net Battery 2 Vin: no longer D6.2 (A)
- net GND: now also U4.13, U4.16, U4.6, U4.7; no longer R3.2, R4.2
- net GNDD: now also C2.2, C3.2, C4.2, C5.2, U4.2, U4.3
- net Solar Charge Battery 2: now also D1.2 (A); no longer D1.1 (K)
- net Solar Charge Battery 2 Switch Sensor: now also C5.1
- net VCC_3V3: now also K5.5, U4.10, U4.11; no longer K5.1, Q5.3 (C), Q6.3 (C)
- net VIN: now also D1.1 (K), D3.1 (K), D4.1 (K); no longer D1.2 (A), D3.2 (A), D4.2 (A)
- net at A2.11 (D8): now also C3.1, U4.12; no longer R8.1
- net at A2.12 (D9): now also C4.1, U4.9; no longer R9.1
- net at A2.13 (D10/CS): now also R8.1
- net at A2.14 (D11/COPI): now also R9.1
- net at D2.2 (A): now also K5.1, Q5.3 (C), Q6.3 (C); no longer K5.5
- net at R8.2: now also U4.1
- net at R9.2: now also U4.4
- new net Battery 2 Vin : D6.2 (A)
- new net Battery Box Fan1 Control: U4.15
- new net Battery Box Fan1 Sensor: R4.2, U4.5
- new net Battery Box Fan2 Control: U4.14
- new net Battery Box Fan2 Sensor: R3.2, U4.8
- no-connect marks 15 -> 11
Other:
- note added: "Battery Box Fan"
- moved on the sheet: C7, C8, D1, D3, D4, D5, D6, Q5, Q6, R13, R17, R5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
