File: electrical/campervan_management/campervan_management.kicad_sch (KiCad schematic)
At the start: 88 parts, among them J1 Duoetto Remote, J2 Input Flow Sensor, J3 Output Flow Sensor, J4 Battery Box, J5 Starter Battery, J6 Fuse and Switch Box, J7 Fuse and Switch, J8 Lights, K2 G5Q-1, K3 G5Q-1, Q1 2N2222, Q2 D4184, Q3 2N2222, Q4 2N2222, Q5 D4184, SW1 SW_Push, U1 RS485-TTL, U2 LM7805, U3 MCP6004, U4 PC817, U5 DS18B20, U6 MCP6001U, U7 PC817

Commit message: First attempt at PCB design
Parts:
- removed C1: 0.33uF, Capacitor_THT:CP_Radial_Tantal_D5.0mm_P5.00mm, symbol Device:C_Polarized_Small_US
- removed C11, C12, C3, C4, C5, C6: 1uF, symbol Device:C
- removed C2: 0.1uF, Capacitor_THT:CP_Radial_Tantal_D5.0mm_P5.00mm, symbol Device:C_Polarized_Small_US
- removed D5, D6: 1N914, Diode_THT:D_DO-35_SOD27_P7.62mm_Horizontal, symbol Diode:1N914
- removed D7, D8: 1N4001, Diode_THT:D_DO-41_SOD81_P10.16mm_Horizontal, symbol Diode:1N4001
- removed J1: Duoetto Remote, Connector_Molex:Molex_Mini-Fit_Jr_5569-02A1_2x01_P4.20mm_Horizontal, symbol Connector:Conn_01x02_Pin
- removed J4: Battery Box, Connector_Molex:Molex_Mini-Fit_Jr_5569-16A2_2x08_P4.20mm_Horizontal, symbol Connector:Conn_01x16_Pin
- removed J5: Starter Battery, Connector_Molex:Molex_Mini-Fit_Jr_5569-02A2_2x01_P4.20mm_Horizontal, symbol Connector:Conn_01x01_Pin
- removed J6: Fuse and Switch Box, Connector_Molex:Molex_Mini-Fit_Jr_5569-06A1_2x03_P4.20mm_Horizontal, symbol Connector:Conn_01x06_Pin
- removed J7: Fuse and Switch, Connector_Molex:Molex_Mini-Fit_Jr_5569-02A1_2x01_P4.20mm_Horizontal, symbol Connector:Conn_01x02_Pin
- removed J8: Lights, Connector_Molex:Molex_Mini-Fit_Jr_5569-02A1_2x01_P4.20mm_Horizontal, symbol Connector:Conn_01x02_Pin
- removed K2, K3: G5Q-1, Relay_THT:Relay_SPDT_Omron-G5Q-1, symbol Relay:G5Q-1
- removed Q1, Q3, Q4: 2N2222, Package_TO_SOT_THT:TO-18-3, symbol Transistor_BJT:BC107
- removed Q2, Q5: D4184, symbol Simulation_SPICE:NMOS
- removed R43: 10k, symbol Device:R
- removed R44, R45: 154k, symbol Device:R
- removed R46: 35.7K 1%, Resistor_THT:R_Axial_DIN0207_L6.3mm_D2.5mm_P10.16mm_Horizontal, symbol Device:R
- removed R47: 10K 1%, Resistor_THT:R_Axial_DIN0207_L6.3mm_D2.5mm_P10.16mm_Horizontal, symbol Device:R
- removed U1: RS485-TTL, Package_SO:SOIC-8_3.9x4.9mm_P1.27mm, symbol Interface_UART:ISL3178E
- removed U2: LM7805, Package_TO_SOT_THT:TO-220-3_Vertical, symbol Regulator_Linear:LM7805_TO220
- removed U3: MCP6004, symbol Amplifier_Operational:MCP6004
- removed U4, U7: PC817, Package_DIP:DIP-4_W7.62mm, symbol Isolator:PC817
- removed U5: DS18B20, Package_TO_SOT_THT:TO-92_Inline, symbol Sensor_Temperature:DS18B20
- removed U6: MCP6001U, symbol Amplifier_Operational:MCP6001U
- added A2: MAX485, CV_connector:RS485_MODULE, symbol camper_van:MAX485_module
- added C1, C10, C11, C2, C22, C25, C27, C3, C4, C5, C6, C7, C8, C9: 100nF, Capacitor_THT:C_Disc_D3.8mm_W2.6mm_P2.50mm, symbol Device:C_Small
- added C12, C13: 0.33uF, Capacitor_THT:C_Disc_D5.0mm_W2.5mm_P2.50mm, symbol Device:C_Polarized_Small_US
- added C18, C19, C21, C24, C26: 1uF, CV_capacitor:CAP_NP_5X11_MTC, symbol Device:C
- added C20: 0.1uF, Capacitor_THT:CP_Radial_Tantal_D5.0mm_P5.00mm, symbol Device:C_Polarized_Small_US
- added C23: 22uF, Capacitor_THT:CP_Radial_Tantal_D4.5mm_P2.50mm, symbol Device:C_Polarized_Small_US
- added D2: 1N914, Diode_THT:D_DO-35_SOD27_P7.62mm_Horizontal, symbol Diode:1N914
- added D5, D6: 1N4001, Diode_THT:D_DO-41_SOD81_P10.16mm_Horizontal, symbol Diode:1N4001
- added J1: Fans, Connector_Molex:Molex_Mini-Fit_Jr_5566-04A_2x02_P4.20mm_Vertical, symbol Connector:Conn_01x04_Socket
- added J10: Starter Battery, Connector_Molex:Molex_Mini-Fit_Jr_5566-02A_2x01_P4.20mm_Vertical, symbol Connector:Conn_01x02_Socket
- added J11: Battery & Fuse, Connector_Molex:Molex_Mini-Fit_Jr_5566-04A_2x02_P4.20mm_Vertical, symbol Connector:Conn_01x04_Socket
- added J4: Battery 2, Connector_Molex:Molex_Mini-Fit_Jr_5566-04A_2x02_P4.20mm_Vertical, symbol Connector:Conn_01x04_Socket
- added J5: Power On/Off, Connector_Molex:Molex_Mini-Fit_Jr_5566-02A_2x01_P4.20mm_Vertical, symbol Connector:Conn_01x02_Socket
- added J6: Temp, Connector_PinSocket_2.54mm:PinSocket_1x03_P2.54mm_Vertical, symbol Connector:Conn_01x03_Socket
- added J7: 12V Power, Connector_Molex:Molex_Mini-Fit_Jr_5566-02A_2x01_P4.20mm_Vertical, symbol Connector:Conn_01x02_Socket
- added J8: Relays, Connector_Molex:Molex_Mini-Fit_Jr_5566-04A_2x02_P4.20mm_Vertical, symbol Connector:Conn_01x04_Socket
- added J9: RS485, Connector_Molex:Molex_Mini-Fit_Jr_5566-02A_2x01_P4.20mm_Vertical, symbol Connector:Conn_01x02_Socket
- added K1: G5V-1, Relay_THT:Relay_SPDT_Omron-G5Q-1, symbol Relay:G5Q-1
- added Q1, Q2, Q3, Q4: STP40NF30L, Package_TO_SOT_THT:TO-220F-3_Vertical, symbol camper_van:STP40NF03L
- added Q5, Q6: 2N2222, Package_TO_SOT_THT:TO-18-3, symbol Transistor_BJT:BC107
- added R14: 41R 2W, Resistor_THT:R_Axial_DIN0414_L11.9mm_D4.5mm_P25.40mm_Horizontal, symbol Device:R
- added R15: 680, Resistor_THT:R_Axial_DIN0207_L6.3mm_D2.5mm_P10.16mm_Horizontal, symbol Device:R
- added U1, U2: ILQ615-3, Package_DIP:DIP-16_W7.62mm, symbol camper_van:ILQ615-3
- added U10, U11, U9: IL300, Package_DIP:DIP-8_W7.62mm, symbol Isolator_Analog:IL300
- added U12, U5: MCP6004, Package_DIP:DIP-14_W7.62mm, symbol Amplifier_Operational:MCP6004
- added U3: CNY17-3, Package_DIP:DIP-6_W7.62mm, symbol Isolator:CNY17-3
- added U4: DS18B20, Package_TO_SOT_THT:TO-92_Inline, symbol Sensor_Temperature:DS18B20
- added U6: MCP6002-xP, Package_DIP:DIP-8_W7.62mm, symbol Amplifier_Operational:MCP6002-xP
- added U7: LM7805, Package_TO_SOT_THT:TO-220-3_Vertical, symbol Regulator_Linear:LM7805_TO220
- added U8: BA00, Package_TO_SOT_THT:TO-220-5_P3.4x3.8mm_StaggerOdd_Lead7.13mm_TabDown, symbol camper_van:BA00
- C14: renamed from C9; footprint (none) -> CV_capacitor:CAP_NP_5X11_MTC
- C15: renamed from C10; footprint (none) -> CV_capacitor:CAP_NP_5X11_MTC
- C16: renamed from C7; footprint (none) -> CV_capacitor:CAP_NP_5X11_MTC
- C17: renamed from C8; footprint (none) -> CV_capacitor:CAP_NP_5X11_MTC
- J2, J3: footprint Connector_Molex:CONN_SD-172648-0000_02_MOL -> Connector_PinSocket_2.54mm:PinSocket_1x03_P2.54mm_Vertical
- R1: value 150 -> 100 2W; footprint Resistor_THT:R_Axial_DIN0207_L6.3mm_D2.5mm_P10.16mm_Horizontal -> Resistor_THT:R_Axial_DIN0414_L11.9mm_D4.5mm_P25.40mm_Horizontal
- R10, R8: value 10K 1% -> 180
- R11: value 35.7K 1% -> 4k7
- R12: value 10K 1% -> 4k7
- R16: value 150 -> 680
- R17: value 35.7K 1% -> 150
- R18: value 10K 1% -> 5k9
- R19, R21, R41: value 4k7 -> 10k; footprint (none) -> Resistor_THT:R_Axial_DIN0207_L6.3mm_D2.5mm_P10.16mm_Horizontal
- R2: value 1k -> 1M; footprint (none) -> Resistor_THT:R_Axial_DIN0207_L6.3mm_D2.5mm_P10.16mm_Horizontal
- R20: value 100 -> 5k9; footprint (none) -> Resistor_THT:R_Axial_DIN0207_L6.3mm_D2.5mm_P10.16mm_Horizontal
- R22, R23, R24, R25, R26, R30, R31: footprint (none) -> Resistor_THT:R_Axial_DIN0207_L6.3mm_D2.5mm_P10.16mm_Horizontal
- R27: value 154k -> 68k; footprint (none) -> Resistor_THT:R_Axial_DIN0207_L6.3mm_D2.5mm_P10.16mm_Horizontal
- R28, R42: value 5k9 -> 10k; footprint (none) -> Resistor_THT:R_Axial_DIN0207_L6.3mm_D2.5mm_P10.16mm_Horizontal
- R29: value 10k -> 154k; footprint (none) -> Resistor_THT:R_Axial_DIN0207_L6.3mm_D2.5mm_P10.16mm_Horizontal
- R3: value 35.7K 1% -> 47k
- R32: value 5k9 -> 22k; footprint (none) -> Resistor_THT:R_Axial_DIN0207_L6.3mm_D2.5mm_P10.16mm_Horizontal
- R33: value 10k -> 22k; footprint (none) -> Resistor_THT:R_Axial_DIN0207_L6.3mm_D2.5mm_P10.16mm_Horizontal
- R34: value 154k -> 22k; footprint (none) -> Resistor_THT:R_Axial_DIN0207_L6.3mm_D2.5mm_P10.16mm_Horizontal
- R35: value 154k -> 1k2; footprint (none) -> Resistor_THT:R_Axial_DIN0207_L6.3mm_D2.5mm_P10.16mm_Horizontal
- R36: value 5k9 -> 1k2; footprint (none) -> Resistor_THT:R_Axial_DIN0207_L6.3mm_D2.5mm_P10.16mm_Horizontal
- R37: value 10k -> 1k2; footprint (none) -> Resistor_THT:R_Axial_DIN0207_L6.3mm_D2.5mm_P10.16mm_Horizontal
- R38: value 1k -> 100k; footprint (none) -> Resistor_THT:R_Axial_DIN0207_L6.3mm_D2.5mm_P10.16mm_Horizontal
- R39: value 4k7 -> 100k; footprint (none) -> Resistor_THT:R_Axial_DIN0207_L6.3mm_D2.5mm_P10.16mm_Horizontal
- R4: value 10K 1% -> 47k
- R40: value 100 -> 100k; footprint (none) -> Resistor_THT:R_Axial_DIN0207_L6.3mm_D2.5mm_P10.16mm_Horizontal
- R5, R7: value 35.7K 1% -> 680
- R6: value 10K 1% -> 2k2
- R9: value 35.7K 1% -> 180
- SW1: footprint Button_Switch_SMD:SW_SPST_EVQP2 -> Button_Switch_THT:SW_TH_Tactile_Omron_B3F-102x
Connections:
- net +12V: now also R3.1, R4.1, J7.2 (Pin_2), U10.2, U11.2, U3.5, U9.2; no longer D1.1 (K), R21.1, R39.1
- net Battery 2 On/Off: now also A1.22 (A3), R17.1; no longer A1.13 (D10/CS), R16.1
- net Battery 2 On/Off Switch Sensor: now also A1.6 (D3), R13.1, C2.1, U2.16; no longer A1.12 (D9), R17.2, R18.1
- net GND: now also R11.2, R2.2, R28.2, R42.2, A2.5 (GND), C12.2, C13.2, C20.2, C23.2, C26.2, C27.2, J10.1 (Pin_1), J4.4 (Pin_4), J5.1 (Pin_1), J6.3 (Pin_3), J7.1 (Pin_1), Q1.3 (S), Q2.3 (S), Q4.3 (S), U1.13, U1.16, U1.6, U1.7, U10.4, U11.4, U12.11 (V-), U12.13 (-), U2.2, U2.3, U2.6, U2.7, U4.1 (GND), U6.2 (-), U6.6 (-), U7.2 (GND), U8.1 (CTL), U8.3 (GND), U9.4; no longer A1.29 (GND), A1.4 (GND), C15.2, C17.2, R10.2, R18.2, R19.2, R23.2, R29.2, R33.2, R37.2, R4.2, R41.2, R8.2, SW1.2
- net Input Flow Sensor: now also A1.15 (D12/CIPO); no longer A1.10 (D7)
- net Output Flow Sensor: now also A1.16 (D13/SCK); no longer A1.11 (D8)
- net VIN: now also D1.1 (K), C13.1, D5.1 (K), D6.1 (K), J4.2 (Pin_2), J8.2 (Pin_2), U8.2 (VIN); no longer A1.30 (VIN)
- net at R24.2: now also C15.1, U5.3 (+); no longer R25.1
- net at R22.1: now also A1.21 (A2), C18.2, C9.1, U12.1; no longer A1.22 (A3)
- net at R40.1: now also J10.2 (Pin_2)
- net at R40.2: now also U11.3, U12.12 (+); no longer R41.1
- net at R38.2: now also U6.3 (+), U9.3
- net at R39.2: now also U10.3, U6.5 (+)
- net at R32.2: now also R29.1, U5.7; no longer R33.1
- net Battery 2 Fuse Sensor: now reaches R16.2
- net Battery 2 Fuse Sensor: now also J11.4 (Pin_4)
- net at R27.2: now also R28.1, U8.5 (ADJ)
- net at D4.2 (A): now also J8.3 (Pin_3), K1.4
- net at R22.2, R23.1: now also U12.2 (-)
- net at R19.1: now also R18.2, U5.2 (-); no longer R20.2
- net at R35.2: now also U9.1; no longer C15.1
- net at D3.2 (A): now also J8.4 (Pin_4), K1.3
- net at R1.1: now also Q2.2 (D)
- net at A1.19 (A0), C14.2: now also R18.1, C10.1, U5.1; no longer R36.1
- net Solar Charge Battery 2: now reaches R1.2
- net Solar Charge Battery 2: now also D1.2 (A), J8.1 (Pin_1), Q1.2 (D); no longer A1.6 (D3)
- net at C16.1, R30.2: now also R25.1; no longer R31.1
- net at A1.20 (A1), C16.2: now also R20.1, C11.1, U5.14; no longer R32.1
- net at R42.1: now also R41.2, U12.5 (+); no longer A1.23 (SDA/A4)
- net at R2.1: now also C1.1, Q1.1 (G); no longer A1.8 (D5)
- net Tx: now reaches A1.1 (D1/TX)
- net Tx: now also A2.4 (DI)
- net at A1.14 (D11/COPI): now also C3.1, U1.9
- net Rx: now reaches A1.2 (D0/RX)
- net Rx: now also A2.1 (RO)
- net En: now reaches A1.5 (D2)
- net En: now also A2.2 (~{RE}), A2.3 (DE)
- net at R26.2: now also C19.1, U12.3 (+); no longer R27.1
- net at R31.2: now also R26.1, C18.1; no longer C17.1
- net at R36.2: now also U10.1; no longer R37.1
- net GNDA: now reaches R21.2
- net GNDA: now also C15.2, C17.2, R19.2, R23.2, C19.2, C21.2, C22.2, C24.2, C25.2, U10.5, U11.5, U12.9 (-), U5.11 (V-), U5.6 (-), U5.9 (-), U6.4 (V-), U9.5
- net at R25.2: now also C17.1, U5.12 (+)
- net +5V renamed VCC_3V3
- net VCC_3V3: now also R41.1, A2.8 (VCC), C20.1, C21.1, C22.1, C24.1, C25.1, C26.1, C27.1, D2.1 (K), J6.1 (Pin_1), K1.5, U1.10, U1.11, U12.4 (V+), U2.10, U2.11, U2.14, U2.15, U4.3 (V_{DD}), U5.4 (V+), U6.8 (V+), U7.3 (VO)
- net 12V Power On/Off: no longer names the net of R13.2
- net 12V Power On/Off: now also Q5.2 (B); no longer A1.16 (D13/SCK)
- net Battery 1 In Sensor: no longer names the net of R5.1
- net Battery 1 In Sensor: now also U2.1
- net Battery 1 Out Sensor: no longer names the net of R9.1
- net Battery 1 Out Sensor: now also A1.12 (D9)
- net Battery 2 In Sensor: no longer names the net of R7.1
- net Battery 2 In Sensor: now also U2.4
- net Battery 2 Out Sensor: no longer names the net of R11.1
- net Battery 2 Out Sensor: now also C6.1, Q3.1 (G)
- net DS18B20 Temp Sensors: no longer names the net of A1.26 (A7)
- net DS18B20 Temp Sensors: now also J6.2 (Pin_2), U4.2 (DQ)
- net Light Control: no longer names the net of R38.1
- net Light Control: now also D5.2 (A), J11.1 (Pin_1); no longer A1.9 (D6)
- removed net Solar Switch: D1.2 (A), R3.1
- new net: J1.1 (Pin_1), R4.2, U1.8
- new net: A1.11 (D8), R8.1
- new net: A1.13 (D10/CS), C4.1, U1.12
- new net: R16.1, U2.8
- new net: R34.1, U11.6, U12.10 (+)
- new net: R31.1, R34.2, U12.8
- new net: Q4.2 (D), R14.1
- new net: K1.2, Q3.2 (D), R14.2
- new net: D6.2 (A), J11.2 (Pin_2), R39.1
- new net: R15.1, U2.5
- new net: C14.1, R24.1, R29.2
- new net: J1.2 (Pin_2), R3.2, U1.5
- new net: J1.3 (Pin_3), U1.15
- new net: J1.4 (Pin_4), U1.14
- new net: D2.2 (A), K1.1, Q5.3 (C), Q6.3 (C)
- new net: C1.2, J4.3 (Pin_3), Q2.1 (G), R6.1, R7.2, U3.4
- new net: A2.7 (B), J9.1 (Pin_1)
- new net: A2.6 (A), J9.2 (Pin_2)
- new net: R10.2, U3.1
- new net: Q6.2 (B), R17.2
- new net: R35.1, U6.1
- new net: R37.2, U11.1
- new net: R32.1, U5.5 (+), U9.6
- new net: R36.1, U6.7
- new net: R9.2, U1.4
- new net: J5.2 (Pin_2), Q3.3 (S)
- new net: R20.2, R21.1, U5.13 (-)
- new net: R33.1, U10.6, U5.10 (+)
- new net: R30.1, R33.2, U5.8
- new net: R37.1, U12.14
- new net: J4.1 (Pin_1), R5.2
- new net: R8.2, U1.1
- new net: U12.6 (-), U12.7
- new net Batteries On: A1.23 (SDA/A4), C6.2, Q4.1 (G), R12.1
- new net Battery 1 Fuse Digital: A1.8 (D5), C7.1, U2.12
- new net Battery 1 Fuse Sensor: J11.3 (Pin_3), R15.2
- new net Battery 2 Fuse Digital: A1.9 (D6), C8.1, U2.9
- new net GNDD: A1.29 (GND), A1.4 (GND), C10.2, C11.2, C2.2, C3.2, C4.2, C5.2, C7.2, C8.2, C9.2, Q5.1 (E), Q6.1 (E), SW1.2, U1.2, U1.3, U3.2
- new net Solar Charge Battery 2 On: A1.10 (D7), R10.1
- new net Solar Charge Battery 2 Switch Sensor: A1.7 (D4), C5.1, U2.13
- new net VCC_MM_9V5: A1.30 (VIN), C12.1, C23.1, R27.1, U7.1 (VI), U8.4 (VOUT)
- no-connect marks 9 -> 7
Other:
- note added: "Battery 1 Vin"
- note added: "Battery 2 Switch"
- note added: "Battery 2 Vin"
- note added: "Battery Box Fan"
- note added: "Battery Box Fan1 Control"
- note added: "Battery Box Fan1 Sensor"
- note added: "Battery Box Fan2 Control"
- note added: "Battery Box Fan2 Sensor"
- note removed: "12V Power On/Off"
- note removed: "Battery 2 On/Off"
- note removed: "Solar/50A charge Battery 2"
- moved on the sheet: C14, C15, C16, C17

Commit message: updates
Parts:
- removed J7: 12V Power, Connector_Molex:Molex_Mini-Fit_Jr_5566-02A_2x01_P4.20mm_Vertical, symbol Connector:Conn_01x02_Socket
- removed U12: MCP6004, Package_DIP:DIP-14_W7.62mm, symbol Amplifier_Operational:MCP6004
- added C28: 1uF, CV_capacitor:CAP_NP_5X11_MTC, symbol Device:C
- added C29: 100nF, Capacitor_THT:C_Disc_D3.8mm_W2.6mm_P2.50mm, symbol Device:C_Small
- added C30: 0.33uF, Capacitor_THT:C_Disc_D5.0mm_W2.5mm_P2.50mm, symbol Device:C_Polarized_Small_US
- added C31: 0.1uF, Capacitor_THT:CP_Radial_Tantal_D5.0mm_P5.00mm, symbol Device:C_Polarized_Small_US
- added R43, R44, R45: 357k, Resistor_THT:R_Axial_DIN0207_L6.3mm_D2.5mm_P10.16mm_Horizontal, symbol Device:R
- added U13, U14: MCP6002-xP, Package_DIP:DIP-8_W7.62mm, symbol Amplifier_Operational:MCP6002-xP
- added U8: LP2950-3.3_TO92, Package_TO_SOT_THT:TO-92_Inline, symbol Regulator_Linear:LP2950-3.3_TO92
- renumbered A2 to A1, A1 to A2, C13 to C1, C7 to C10, C3 to C11, C8 to C12, C11 to C13, C9 to C14, C10 to C15, C18 to C16, C19 to C17, C27 to C18, C26 to C19, C12 to C2, C21 to C20, C22 to C21, C15 to C22, C14 to C23, C16 to C26, C17 to C27, C23 to C3, C20 to C4, C1 to C5, C2 to C7, C5 to C8, C4 to C9, D5 to D1, D4 to D2, D6 to D4, D2 to D5, D1 to D6, J4 to J1, J2 to J10, J10 to J11, J11 to J3, J5 to J4, J8 to J5, J9 to J7, J1 to J8, J3 to J9, Q5 to Q1, Q1 to Q3, Q6 to Q4, Q4 to Q5, Q3 to Q6, R2 to R1, R11 to R10, R1 to R11, R6 to R12, R10 to R13, R16 to R14, R8 to R15, R14 to R16, R4 to R17, R3 to R18, R9 to R19, R27 to R2, R31 to R20, R22 to R21, R23 to R22, R41 to R23, R26 to R24, R40 to R25, R37 to R26, R34 to R27, R38 to R28, R39 to R29, R28 to R3, R35 to R30, R36 to R31, R24 to R32, R18 to R33, R19 to R34, R20 to R35, R21 to R36, R30 to R37, R29 to R38, R25 to R39, R7 to R4, R42 to R40, R32 to R41, R33 to R42, R15 to R6, R17 to R7, R13 to R8, R12 to R9, U7 to U1, U6 to U10, U10 to U11, U5 to U12, U8 to U2, U2 to U3, U3 to U4, U1 to U5, U4 to U6, U11 to U7
Connections:
- net GNDA is gone; now on net GND: C17.2, C20.2, C21.2, C22.2, C24.2, C25.2, C27.2, R22.2, R34.2, R36.2, U10.4 (V-), U11.5, U12.11 (V-), U12.6 (-), U12.9 (-), U7.5, U9.5
- net GNDD is gone; now on net GND: A2.29 (GND), A2.4 (GND), C10.2, C11.2, C12.2, C13.2, C14.2, C15.2, C7.2, C8.2, C9.2, Q1.1 (E), Q4.1 (E), SW1.2, U4.2, U5.2, U5.3
- net GND: now also C28.2, C29.2, C30.2, C31.2, R43.2, R44.2, R45.2, U13.4 (V-), U13.6 (-), U14.2 (-), U14.4 (V-), U8.2 (GND)
- net VCC_3V3: no longer C18.1, C19.1, C20.1, C21.1, C24.1, C25.1, R23.1, U10.8 (V+), U12.4 (V+)
- net VCC_MM_9V5: now also C30.1, U8.3 (VI)
- net VIN: now also R17.1, R18.1, U4.5
- net at A2.21 (A2), C14.1, C16.2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: now also U13.1
- net at R27.1, U7.6: now also U13.5 (+)
- net at R20.1, R27.2: now also U13.7
- net at R21.2, R22.1: now also U13.2 (-)
- net at R29.2, U10.5 (+), U11.3: now also R43.1
- net at C17.1, R24.2: now also U13.3 (+)
- net at R25.2, U7.3: now also R44.1, U14.3 (+)
- net at R28.2, U10.3 (+), U9.3: now also R45.1
- net at R26.1: now also U14.1
- net at R23.2, R40.1: now also U14.5 (+)
- net +12V renamed VCC_3V3A
- net VCC_3V3A: now also C18.1, C19.1, C20.1, C21.1, C24.1, C25.1, R23.1, U10.8 (V+), U12.4 (V+), C28.1, C29.1, C31.1, U13.8 (V+), U14.8 (V+), U8.1 (VO); no longer R17.1, R18.1, U4.5
- new net: U14.6 (-), U14.7
Other:
- moved on the sheet: A1, C1, C10, C12, C18, C19, C2, C20, C21, C24, C25, C3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
