File: electrical/campervan_management_V2/_autosave-campervan_management_V2.kicad_pcb (KiCad board)
At the start: 4 copper layers, 140 x 95 mm, 163 parts, among them J1 Battery & Fuse, J10 RS485, J11 Power On/Off Switch, J2 Battery 2, J3 Relays, J5 Input Flow Sensor, J6 Temp, J7 Output Flow Sensor, J8 Starter Battery, J9 Fans, K1 G6KU-2, Q1 Q_PMOS_DGS, Q10 Q_PMOS_DGS, Q2 Q_PMOS_DGS, Q4 MMBT2222A, Q6 MMBT2222A, Q7 Q_PMOS_DGS, Q8 Q_PMOS_DGS, Q9 Q_PMOS_DGS, SW1 SW_Push, U1 MCP16311T-E/MNS, U10 LM358DR2G, U11 LM358DR2G, U12 LTV-817S-TA1-C, U13 LTV-817S-TA1-C, U14 HCNR200-500E, U15 LM358DR2G, U16 LTV-817S-TA1-C, U17 LTV-817S-TA1-C, U18 LTV-817S-TA1-C, U19 MAX487E, U2 AMS1117-3.3, U20 LTV-817S-TA1-C, U21 LTV-817S-TA1-C, U22 LTV-817S-TA1-C, U23 LTV-817S-TA1-C, U24 LTV-817S-TA1-C, U25 MCP16311T-E/MNS, U3 LTV-817S-TA1-C, U4 HCNR200-500E, U5 AMS1117-3.3, U6 LM358DR2G, U7 LM358DR2G, U8 LTV-817S-TA1-C, U9 HCNR200-500E

Commit message: updated
Parts:
- R12, R35, R7: value 10k -> 220k
- R19, R24, R40: value 120k -> 10k; footprint Resistor_SMD:R_0603_1608Metric -> Potentiometer_THT:Potentiometer_Bourns_3296W_Vertical
- moved J6 62.2 mm to (138.6, 77.2)
- moved J7 62.2 mm to (143.2, 77.2)
- moved J5 61.5 mm to (134.2, 77.1)
- moved R40 21.5 mm to (171.9, 136.7), turned to 0 degrees
- moved R24 20.9 mm to (174.0, 108.3), turned to 0 degrees
- moved R19 19.3 mm to (173.8, 122.8)
Connections:
- R12 pad 2: Net-(U7A-+) -> Net-(U7A--)
- R16 pad 1: Net-(U6B-+) -> Net-(R16-Pad1)
- R19 pad 1: Net-(U7B-+) -> Net-(R19-Pad1)
- R19 pad 2: GND -> Net-(U10B--)
- R24 pad 1: Net-(U7A-+) -> Net-(R16-Pad1)
- R24 pad 2: GND -> Net-(U6B--)
- R28 pad 1: Net-(U10B-+) -> Net-(R19-Pad1)
- R35 pad 2: Net-(U11A-+) -> Net-(U11A--)
- R40 pad 1: Net-(U11A-+) -> Net-(R40-Pad1)
- R40 pad 2: GND -> Net-(U15B--)
- R46 pad 1: Net-(U15B-+) -> Net-(R40-Pad1)
- R7 pad 2: Net-(U7B-+) -> Net-(U7B--)
- U10 pad 5: Net-(U10B-+) -> GND
- U10 pad 6: GND -> Net-(U10B--)
- U11 pad 2: GND -> Net-(U11A--)
- U11 pad 3: Net-(U11A-+) -> GND
- U14 pad 3: Net-(U11A-+) -> Net-(U11A--)
- U14 pad 6: Net-(U15B-+) -> Net-(U15B--)
- U15 pad 5: Net-(U15B-+) -> GND
- U15 pad 6: GND -> Net-(U15B--)
- U4 pad 3: Net-(U7B-+) -> Net-(U7B--)
- U4 pad 6: Net-(U6B-+) -> Net-(U6B--)
- U6 pad 5: Net-(U6B-+) -> GND
- U6 pad 6: GND -> Net-(U6B--)
- U7 pad 2: GND -> Net-(U7A--)
- U7 pad 3: Net-(U7A-+) -> GND
- U7 pad 5: Net-(U7B-+) -> GND
- U7 pad 6: GND -> Net-(U7B--)
- U9 pad 3: Net-(U7A-+) -> Net-(U7A--)
- U9 pad 6: Net-(U10B-+) -> Net-(U10B--)
Routing:
- net Net-(U15B-+): track 10.6 -> 0.00 mm
- net Net-(U11A-+): track 10.5 -> 0.00 mm
- net (no net): track 0.00 -> 10.5 mm
- net Net-(U6B-+): track 2.08 -> 0.00 mm
- net Net-(U7A-+): track 1.78 -> 0.00 mm
- net Net-(U7B-+): track 1.72 -> 0.00 mm
- net Net-(U10B-+): track 1.72 -> 0.00 mm
