File: electrical/campervan_management_V2/campervan_management_V2.kicad_sch (KiCad schematic)
At the start: 22 parts, among them J1 Battery & Fuse, J2 RS485, J3 Temp, J4 Output Flow Sensor, J5 Input Flow Sensor, J6 Power On/Off Switch, J7 Starter Battery, J8 Battery 2, J9 Relays, SW1 SW_Push, U5 MAX487E

Commit message: Close to final design
Parts:
- removed J8: Battery 2, Connector_Molex:Molex_Mini-Fit_Jr_5566-04A_2x02_P4.20mm_Vertical, symbol Connector:Conn_01x04_Socket
- added J2: Battery 2, Connector_Molex:Molex_Mini-Fit_Jr_5566-02A_2x01_P4.20mm_Vertical, symbol Connector:Conn_01x02_Socket
- added J3: Solar Charge, Connector_Molex:Molex_Mini-Fit_Jr_5566-02A_2x01_P4.20mm_Vertical, symbol Connector:Conn_01x02_Socket
- U8: renamed from U5; JLCPCB (none) -> 1.67; e14 (none) -> 12
- renumbered C40 to C26, C44 to C27, C47 to C28, H4 to H3, H3 to H4, J4 to J10, J5 to J11, J6 to J4, J2 to J5, J9 to J7, J3 to J8, J7 to J9, R8 to R16, R9 to R17, R10 to R18
Connections:
- net Batteries On: now also A1.12 (D9); no longer A1.23 (SDA/A4)
- net Battery 2 On/Off: now also A1.13 (D10/CS); no longer A1.22 (A3)
- net Battery Box Fan1 Control: now also A1.24 (SCL/A5); no longer A1.13 (D10/CS)
- net Battery Box Fan1 Sensor: now also A1.23 (SDA/A4); no longer A1.11 (D8)
- net Battery Box Fan2 Control: now also A1.25 (A6); no longer A1.14 (D11/COPI)
- net Battery Box Fan2 Sensor: now also A1.22 (A3); no longer A1.10 (D7)
- net Battery Fuse Sensors/Battery 1 Fuse Sensor: now also J1.4 (Pin_4); no longer J1.1 (Pin_1)
- net Battery Management/Battery 2 Switch: now also J2.1 (Pin_1)
- net Battery Voltage Measurement/Battery 1 Vin: now also J1.1 (Pin_1); no longer J1.4 (Pin_4)
- net Battery Voltage Measurement/Battery 2 Voltage: now also A1.19 (A0), C28.1; no longer A1.21 (A2), C26.1
- net Battery Voltage Measurement/Starter Battery Voltage: now also A1.21 (A2), C26.1; no longer A1.19 (A0), C28.1
- net GND: now also J3.2 (Pin_2)
- net Power Supply Control: now also A1.14 (D11/COPI); no longer A1.24 (SCL/A5)
- net Solar Charge Management/Solar Charge Battery 2 On: now also A1.11 (D8); no longer A1.12 (D9)
- net Solar Charge Management/Solar Charge Battery 2 Switch: now also J3.1 (Pin_1)
- net VIN: now also J2.2 (Pin_2)
Other:
- moved on the sheet: C26

Commit message: Added optocouplers to flow sensors
Parts:
- removed J10: Output Flow Sensor, Connector_Molex:Molex_Mini-Fit_Jr_5566-04A_2x02_P4.20mm_Vertical, symbol Connector:Conn_01x04_Socket
- removed J11: Input Flow Sensor, Connector_Molex:Molex_Mini-Fit_Jr_5566-04A_2x02_P4.20mm_Vertical, symbol Connector:Conn_01x04_Socket
Connections:
- no-connect marks 8 -> 6
Other:
- added sheet Flow Sensors (flow_sensors.kicad_sch)
