File: electrical/campervan_management_V2/3V3_ldo.kicad_sch (KiCad schematic)
At the start: 4 parts, among them U2 AMS1117-3.3

Commit message: Close to final design
Parts:
- U5: renamed from U2; value AMS1117-3.3 -> AMS1117-3.3/TLV761
- renumbered C5 to C15, C3 to C17, C7 to C18
Changed lines of the file:
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@@
 		(dnp no)
 		(fields_autoplaced yes)
-		(property "Reference" "C5"
+		(property "Reference" "C15"
 			(at 109.22 96.5262 0)
 			(effects
@@
 		)
 		(property "Extended" "B"
+			(at 106.68 97.79 0)
+			(effects
+				(font
+					(size 1.27 1.27)
+				)
+				(hide yes)
+			)
+		)
+		(property "JLCPCB" ""
+			(at 106.68 97.79 0)
+			(effects
+				(font
+					(size 1.27 1.27)
+				)
+				(hide yes)
+			)
+		)
+		(property "e14" ""
+			(at 106.68 97.79 0)
+			(effects
+				(font
+					(size 1.27 1.27)
+				)
+				(hide yes)
+			)
+		)
+		(property "Component Class" ""
 			(at 106.68 97.79 0)
 			(effects
@@
 			(project "campervan_management_V2"
 				(path "/870a08cc-a6e6-4310-b4b3-ae6af01530aa/d6c26a68-5132-41c9-800c-60e2b42b3e90/af2552d0-9fb4-47ca-97f2-e4c8a0326568"
-					(reference "C9")
+					(reference "C36")
 					(unit 1)
 				)
 				(path "/870a08cc-a6e6-4310-b4b3-ae6af01530aa/d6c26a68-5132-41c9-800c-60e2b42b3e90/bc027ce7-791c-49ac-a4a6-c15c61794209"
-					(reference "C5")
+					(reference "C15")
 					(unit 1)
 				)
@@
 		(dnp no)
 		(fields_autoplaced yes)
-		(property "Reference" "C3"
+		(property "Reference" "C17"
 			(at 138.43 96.0881 0)
 			(effects
@@
 		)
 		(property "Extended" "B"
+			(at 135.89 97.79 0)
+			(effects
+				(font
+					(size 1.27 1.27)
+				)
+				(hide yes)
+			)
+		)
+		(property "JLCPCB" ""
+			(at 135.89 97.79 0)
+			(effects
+				(font
+					(size 1.27 1.27)
+				)
+				(hide yes)
+			)
+		)
+		(property "e14" ""
+			(at 135.89 97.79 0)
+			(effects
+				(font
+					(size 1.27 1.27)
+				)
+				(hide yes)
+			)
+		)
+		(property "Component Class" ""
 			(at 135.89 97.79 0)
 			(effects
@@
 			(project "campervan_management_V2"
 				(path "/870a08cc-a6e6-4310-b4b3-ae6af01530aa/d6c26a68-5132-41c9-800c-60e2b42b3e90/af2552d0-9fb4-47ca-97f2-e4c8a0326568"
-					(reference "C10")
+					(reference "C38")
 					(unit 1)
 				)
 				(path "/870a08cc-a6e6-4310-b4b3-ae6af01530aa/d6c26a68-5132-41c9-800c-60e2b42b3e90/bc027ce7-791c-49ac-a4a6-c15c61794209"
-					(reference "C3")
+					(reference "C17")
 					(unit 1)
 				)
@@
 		(dnp no)
 		(fields_autoplaced yes)
-		(property "Reference" "C7"
+		(property "Reference" "C18"
 			(at 148.59 96.0881 0)
 			(effects
@@
 		)
 		(property "Extended" "B"
+			(at 146.05 97.79 0)
+			(effects
+				(font
+					(size 1.27 1.27)
+				)
+				(hide yes)
+			)
+		)
+		(property "JLCPCB" ""
+			(at 146.05 97.79 0)
+			(effects
+				(font
+					(size 1.27 1.27)
+				)
+				(hide yes)
+			)
+		)
+		(property "e14" ""
+			(at 146.05 97.79 0)
+			(effects
+				(font
+					(size 1.27 1.27)
+				)
+				(hide yes)
+			)
+		)
+		(property "Component Class" ""
 			(at 146.05 97.79 0)
 			(effects
@@
 			(project "campervan_management_V2"
 				(path "/870a08cc-a6e6-4310-b4b3-ae6af01530aa/d6c26a68-5132-41c9-800c-60e2b42b3e90/af2552d0-9fb4-47ca-97f2-e4c8a0326568"
-					(reference "C6")
+					(reference "C37")
 					(unit 1)
 				)
 				(path "/870a08cc-a6e6-4310-b4b3-ae6af01530aa/d6c26a68-5132-41c9-800c-60e2b42b3e90/bc027ce7-791c-49ac-a4a6-c15c61794209"
-					(reference "C7")
+					(reference "C18")
 					(unit 1)
 				)
@@
 		(dnp no)
 		(fields_autoplaced yes)
-		(property "Reference" "U2"
+		(property "Reference" "U5"
 			(at 121.92 87.63 0)
 			(effects
@@
 			)
 		)
-		(property "Value" "AMS1117-3.3"
+		(property "Value" "AMS1117-3.3/TLV761"
 			(at 121.92 90.17 0)
 			(effects
@@
 		)
 		(property "Extended" "B"
+			(at 121.92 93.98 0)
+			(effects
+				(font
+					(size 1.27 1.27)
+				)
+				(hide yes)
+			)
+		)
+		(property "JLCPCB" ""
+			(at 121.92 93.98 0)
+			(effects
+				(font
+					(size 1.27 1.27)
+				)
+				(hide yes)
+			)
+		)
+		(property "e14" ""
+			(at 121.92 93.98 0)
+			(effects
+				(font
+					(size 1.27 1.27)
+				)
+				(hide yes)
+			)
+		)
+		(property "Component Class" ""
 			(at 121.92 93.98 0)
 			(effects
@@
 			(project "campervan_management_V2"
 				(path "/870a08cc-a6e6-4310-b4b3-ae6af01530aa/d6c26a68-5132-41c9-800c-60e2b42b3e90/af2552d0-9fb4-47ca-97f2-e4c8a0326568"
-					(reference "U4")
+					(reference "U22")
 					(unit 1)
 				)
 				(path "/870a08cc-a6e6-4310-b4b3-ae6af01530aa/d6c26a68-5132-41c9-800c-60e2b42b3e90/bc027ce7-791c-49ac-a4a6-c15c61794209"
-					(reference "U2")
-					(unit 1)
-				)
+					(reference "U5")
+					(unit 1)
+				)
