File: electrical/campervan_management_V2/battery_fuses.kicad_sch (KiCad schematic)
At the start: 6 parts, among them U12 LTV-817S-TA1-C, U16 LTV-817S-TA1-C

Commit message: First attempt at PCB layout
Parts:
- renumbered C33 to C35, C34 to C36, R38 to R18, R44 to R23, U16 to U12, U12 to U8
Changed lines of the file:
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@@
 		(on_board yes)
 		(dnp no)
-		(property "Reference" "U16"
+		(property "Reference" "U12"
 			(at 80.01 77.47 0)
 			(effects
@@
 			(project "campervan_management_V2"
 				(path "/870a08cc-a6e6-4310-b4b3-ae6af01530aa/7b6855ec-62ba-489d-a9bd-50cc04116ffb"
-					(reference "U16")
+					(reference "U12")
 					(unit 1)
 				)
@@
 		(on_board yes)
 		(dnp no)
-		(property "Reference" "U12"
+		(property "Reference" "U8"
 			(at 80.01 45.72 0)
 			(effects
@@
 			(project "campervan_management_V2"
 				(path "/870a08cc-a6e6-4310-b4b3-ae6af01530aa/7b6855ec-62ba-489d-a9bd-50cc04116ffb"
-					(reference "U12")
+					(reference "U8")
 					(unit 1)
 				)
@@
 		(dnp no)
 		(fields_autoplaced yes)
-		(property "Reference" "R44"
+		(property "Reference" "R23"
 			(at 93.98 77.47 90)
 			(effects
@@
 			(project "campervan_management_V2"
 				(path "/870a08cc-a6e6-4310-b4b3-ae6af01530aa/7b6855ec-62ba-489d-a9bd-50cc04116ffb"
-					(reference "R44")
+					(reference "R23")
 					(unit 1)
 				)
@@
 		(dnp no)
 		(fields_autoplaced yes)
-		(property "Reference" "R38"
+		(property "Reference" "R18"
 			(at 93.98 45.72 90)
 			(effects
@@
 			(project "campervan_management_V2"
 				(path "/870a08cc-a6e6-4310-b4b3-ae6af01530aa/7b6855ec-62ba-489d-a9bd-50cc04116ffb"
-					(reference "R38")
+					(reference "R18")
 					(unit 1)
 				)
@@
 		(on_board yes)
 		(dnp no)
-		(property "Reference" "C34"
+		(property "Reference" "C36"
 			(at 67.31 93.9862 0)
 			(effects
@@
 			(project "campervan_management_V2"
 				(path "/870a08cc-a6e6-4310-b4b3-ae6af01530aa/7b6855ec-62ba-489d-a9bd-50cc04116ffb"
-					(reference "C34")
+					(reference "C36")
 					(unit 1)
 				)
@@
 		(on_board yes)
 		(dnp no)
-		(property "Reference" "C33"
+		(property "Reference" "C35"
 			(at 67.31 62.2362 0)
 			(effects
@@
 			(project "campervan_management_V2"
 				(path "/870a08cc-a6e6-4310-b4b3-ae6af01530aa/7b6855ec-62ba-489d-a9bd-50cc04116ffb"
-					(reference "C33")
-					(unit 1)
-				)
+					(reference "C35")
+					(unit 1)
+				)

Commit message: Close to final design
Parts:
- renumbered C35 to C22, C36 to C24, R18 to R19, R23 to R21, U12 to U10, U8 to U9
Connections:
- net Net-(R22-Pad1): now reaches R21.1, U10.1
Changed lines of the file:
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@@
+		)
+	)
+	(label "Net-(R22-Pad1)"
+		(at 87.63 83.82 0)
+		(effects
+			(font
+				(size 1.27 1.27)
+			)
+			(justify left bottom)
+		)
+	)
+	(label "Net-(R22-Pad1)"
+		(at 87.63 83.82 0)
+		(effects
+			(font
+				(size 1.27 1.27)
+			)
+			(justify left bottom)
 		)
 	)
@@
 		(on_board yes)
 		(dnp no)
-		(property "Reference" "U12"
+		(property "Reference" "U10"
 			(at 80.01 77.47 0)
 			(effects
@@
 		)
 		(property "Extended" "B"
+			(at 80.01 86.36 0)
+			(effects
+				(font
+					(size 1.27 1.27)
+				)
+				(hide yes)
+			)
+		)
+		(property "JLCPCB" ""
+			(at 80.01 86.36 0)
+			(effects
+				(font
+					(size 1.27 1.27)
+				)
+				(hide yes)
+			)
+		)
+		(property "e14" ""
+			(at 80.01 86.36 0)
+			(effects
+				(font
+					(size 1.27 1.27)
+				)
+				(hide yes)
+			)
+		)
+		(property "Component Class" ""
 			(at 80.01 86.36 0)
 			(effects
@@
 			(project "campervan_management_V2"
 				(path "/870a08cc-a6e6-4310-b4b3-ae6af01530aa/7b6855ec-62ba-489d-a9bd-50cc04116ffb"
-					(reference "U12")
+					(reference "U10")
 					(unit 1)
 				)
@@
 		(on_board yes)
 		(dnp no)
-		(property "Reference" "U8"
+		(property "Reference" "U9"
 			(at 80.01 45.72 0)
 			(effects
@@
 		)
 		(property "Extended" "B"
+			(at 80.01 54.61 0)
+			(effects
+				(font
+					(size 1.27 1.27)
+				)
+				(hide yes)
+			)
+		)
+		(property "JLCPCB" ""
+			(at 80.01 54.61 0)
+			(effects
+				(font
+					(size 1.27 1.27)
+				)
+				(hide yes)
+			)
+		)
+		(property "e14" ""
+			(at 80.01 54.61 0)
+			(effects
+				(font
+					(size 1.27 1.27)
+				)
+				(hide yes)
+			)
+		)
+		(property "Component Class" ""
 			(at 80.01 54.61 0)
 			(effects
@@
 			(project "campervan_management_V2"
 				(path "/870a08cc-a6e6-4310-b4b3-ae6af01530aa/7b6855ec-62ba-489d-a9bd-50cc04116ffb"
-					(reference "U8")
+					(reference "U9")
 					(unit 1)
 				)
@@
 		(dnp no)
 		(fields_autoplaced yes)
-		(property "Reference" "R23"
+		(property "Reference" "R21"
 			(at 93.98 77.47 90)
 			(effects
@@
 		)
 		(property "Extended" "B"
+			(at 93.98 83.82 90)
+			(effects
+				(font
+					(size 1.27 1.27)
+				)
+				(hide yes)
+			)
+		)
+		(property "JLCPCB" ""
+			(at 93.98 83.82 90)
+			(effects
+				(font
+					(size 1.27 1.27)
+				)
+				(hide yes)
+			)
+		)
+		(property "e14" ""
+			(at 93.98 83.82 90)
+			(effects
+				(font
+					(size 1.27 1.27)
+				)
+				(hide yes)
+			)
+		)
+		(property "Component Class" ""
 			(at 93.98 83.82 90)
 			(effects
@@
 			(project "campervan_management_V2"
 				(path "/870a08cc-a6e6-4310-b4b3-ae6af01530aa/7b6855ec-62ba-489d-a9bd-50cc04116ffb"
-					(reference "R23")
+					(reference "R21")
 					(unit 1)
 				)
@@
 		(dnp no)
 		(fields_autoplaced yes)
-		(property "Reference" "R18"
+		(property "Reference" "R19"
 			(at 93.98 45.72 90)
 			(effects
@@
 		)
 		(property "Extended" "B"
+			(at 93.98 52.07 90)
+			(effects
+				(font
+					(size 1.27 1.27)
+				)
+				(hide yes)
+			)
+		)
+		(property "JLCPCB" ""
+			(at 93.98 52.07 90)
+			(effects
+				(font
+					(size 1.27 1.27)
+				)
+				(hide yes)
+			)
+		)
+		(property "e14" ""
+			(at 93.98 52.07 90)
+			(effects
+				(font
+					(size 1.27 1.27)
+				)
+				(hide yes)
+			)
+		)
+		(property "Component Class" ""
 			(at 93.98 52.07 90)
 			(effects
@@
 			(project "campervan_management_V2"
 				(path "/870a08cc-a6e6-4310-b4b3-ae6af01530aa/7b6855ec-62ba-489d-a9bd-50cc04116ffb"
-					(reference "R18")
+					(reference "R19")
 					(unit 1)
 				)
@@
 		(on_board yes)
 		(dnp no)
-		(property "Reference" "C36"
+		(property "Reference" "C24"
 			(at 67.31 93.9862 0)
 			(effects
@@
 		)
 		(property "Extended" "B"
+			(at 69.85 95.25 0)
+			(effects
+				(font
+					(size 1.27 1.27)
+				)
+				(hide yes)
+			)
+		)
+		(property "JLCPCB" ""
+			(at 69.85 95.25 0)
+			(effects
+				(font
+					(size 1.27 1.27)
+				)
+				(hide yes)
+			)
+		)
+		(property "e14" ""
+			(at 69.85 95.25 0)
+			(effects
+				(font
+					(size 1.27 1.27)
+				)
+				(hide yes)
+			)
+		)
+		(property "Component Class" ""
 			(at 69.85 95.25 0)
 			(effects
@@
 			(project "campervan_management_V2"
 				(path "/870a08cc-a6e6-4310-b4b3-ae6af01530aa/7b6855ec-62ba-489d-a9bd-50cc04116ffb"
-					(reference "C36")
+					(reference "C24")
 					(unit 1)
 				)
@@
 		(on_board yes)
 		(dnp no)
-		(property "Reference" "C35"
+		(property "Reference" "C22"
 			(at 67.31 62.2362 0)
 			(effects
@@
 		)
 		(property "Extended" "B"
+			(at 69.85 63.5 0)
+			(effects
+				(font
+					(size 1.27 1.27)
+				)
+				(hide yes)
+			)
+		)
+		(property "JLCPCB" ""
+			(at 69.85 63.5 0)
+			(effects
+				(font
+					(size 1.27 1.27)
+				)
+				(hide yes)
+			)
+		)
+		(property "e14" ""
+			(at 69.85 63.5 0)
+			(effects
+				(font
+					(size 1.27 1.27)
+				)
+				(hide yes)
+			)
+		)
+		(property "Component Class" ""
 			(at 69.85 63.5 0)
 			(effects
@@
 			(project "campervan_management_V2"
 				(path "/870a08cc-a6e6-4310-b4b3-ae6af01530aa/7b6855ec-62ba-489d-a9bd-50cc04116ffb"
-					(reference "C35")
+					(reference "C22")
 					(unit 1)
 				)
