File: electrical/campervan_management_V2/battery_voltage.kicad_sch (KiCad schematic)
At the start: 47 parts, among them U10 LM358DR2G, U11 LM358DR2G, U14 HCNR200-500E, U15 LM358DR2G, U4 HCNR200-500E, U6 LM358DR2G, U7 LM358DR2G, U9 HCNR200-500E

Commit message: updated
Parts:
- added R19, R24, R40: 10k, Potentiometer_THT:Potentiometer_Bourns_3296W_Vertical, symbol Device:R_Variable
- R12, R35, R7: value 27k -> 220k
Connections:
- net GND: now also U10.5 (+), U11.3 (+), U15.5 (+), U6.5 (+), U7.3 (+), U7.5 (+); no longer U10.6 (-), U11.2 (-), U15.6 (-), U6.6 (-), U7.2 (-), U7.6 (-)
- net at R35.2, U14.3: now also U11.2 (-); no longer U11.3 (+)
- net at R7.2, U4.3: now also U7.6 (-); no longer U7.5 (+)
- net at R12.2, U9.3: now also U7.2 (-); no longer U7.3 (+)
- new net: R40.1, R46.1
- new net: R40.2, U14.6, U15.6 (-)
- new net: R24.2, U4.6, U6.6 (-)
- new net: R16.1, R24.1
- new net: R19.2, U10.6 (-), U9.6
- new net: R19.1, R28.1
Other:
- note added: "1Hz Butterworth LP Filter"
- note added: "Isolation Amplifier - 14.4V to 1.1V"
- note added: "Isolation Amplifier K1 = 0.25% - 0.75%. 0.5% typical K3 = 0.85 - 1.15 V_{in typ} = 12.8V V_(out) = 1.1V If = 10mA I_{p1} = K1 x IF_{max} R1 = V_{in} / I_{p1} R2 = R1 x G / K3"
- moved on the sheet: C10, C11, C12, C13, C17, C18, C21, C22, C23, C24, C25, C26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

Commit message: First attempt at PCB layout
Parts:
- added C20, C25, C33, C41, C42, C50: C_Small, Capacitor_SMD:C_0603_1608Metric, symbol Device:C_Small
- added TP1, TP2, TP3: TestPoint, CV_connector:5000, symbol Connector:TestPoint
- C21: renamed from C32; footprint Capacitor_SMD:C_0805_2012Metric -> Capacitor_SMD:C_0603_1608Metric; LCSC PN C28323 -> C15849
- C23: renamed from C31; footprint Capacitor_SMD:C_0805_2012Metric -> Capacitor_SMD:C_0603_1608Metric; LCSC PN C28323 -> C15849
- C27: renamed from C23; footprint Capacitor_SMD:C_0805_2012Metric -> Capacitor_SMD:C_0603_1608Metric; LCSC PN C28323 -> C15849
- C28: renamed from C27; footprint Capacitor_SMD:C_0805_2012Metric -> Capacitor_SMD:C_0603_1608Metric; LCSC PN C28323 -> C15849
- C30: renamed from C26; footprint Capacitor_SMD:C_0805_2012Metric -> Capacitor_SMD:C_0603_1608Metric; LCSC PN C28323 -> C15849
- C31: renamed from C25; footprint Capacitor_SMD:C_0805_2012Metric -> Capacitor_SMD:C_0603_1608Metric; LCSC PN C28323 -> C15849
- C38: renamed from C22; footprint Capacitor_SMD:C_0805_2012Metric -> Capacitor_SMD:C_0603_1608Metric; LCSC PN C28323 -> C15849
- C45: renamed from C18; footprint Capacitor_SMD:C_0805_2012Metric -> Capacitor_SMD:C_0603_1608Metric; LCSC PN C28323 -> C15849
- C48: renamed from C17; footprint Capacitor_SMD:C_0805_2012Metric -> Capacitor_SMD:C_0603_1608Metric; LCSC PN C28323 -> C15849
- C49: renamed from C11; footprint Capacitor_SMD:C_0805_2012Metric -> Capacitor_SMD:C_0603_1608Metric; LCSC PN C28323 -> C15849
- C52: renamed from C10; footprint Capacitor_SMD:C_0805_2012Metric -> Capacitor_SMD:C_0603_1608Metric; LCSC PN C28323 -> C15849
- R21: renamed from R40; symbol Device:R_Variable -> Device:R_Potentiometer
- R36: renamed from R19; symbol Device:R_Variable -> Device:R_Potentiometer
- R52: renamed from R24; symbol Device:R_Variable -> Device:R_Potentiometer
- U10: renamed from U11; footprint Package_SO:OnSemi_Micro8 -> CV_connector:SOIC-8_ONS-L
- U11: renamed from U15; footprint Package_SO:OnSemi_Micro8 -> CV_connector:SOIC-8_ONS-L
- U15: renamed from U9; footprint Package_SO:SOP-8_3.76x4.96mm_P1.27mm -> Package_DIP:SMDIP-8_W11.48mm
- U17: renamed from U10; footprint Package_SO:OnSemi_Micro8 -> CV_connector:SOIC-8_ONS-L
- U19: renamed from U7; footprint Package_SO:OnSemi_Micro8 -> CV_connector:SOIC-8_ONS-L
- U22: renamed from U4; footprint Package_SO:SOP-8_3.76x4.96mm_P1.27mm -> Package_DIP:SMDIP-8_W11.48mm
- U23: renamed from U6; footprint Package_SO:OnSemi_Micro8 -> CV_connector:SOIC-8_ONS-L
- U9: renamed from U14; footprint Package_SO:SOP-8_3.76x4.96mm_P1.27mm -> Package_DIP:SMDIP-8_W11.48mm
- renumbered C29 to C26, C21 to C37, C13 to C46, C12 to C51, R47 to R14, R42 to R16, R37 to R17, R45 to R19, R33 to R20, R41 to R22, R46 to R24, R32 to R25, R35 to R26, R31 to R30, R25 to R32, R27 to R33, R26 to R35, R28 to R39, R12 to R40, R11 to R41, R8 to R43, R21 to R46, R10 to R47, R7 to R48, R15 to R50, R9 to R53, R16 to R55
Connections:
- net at R21.1, R24.1: now also R21.2
- net at U11.6 (-), U9.6: now also R21.3, C20.2; no longer R21.2
- net at R26.2, U10.2 (-), U9.3: now also C25.2
- net at R32.1, R39.2, U17.7: now also C33.1, TP2.1
- net at U22.6, U23.6 (-): now also R52.3, C50.2; no longer R52.2
- net at R47.1, R55.2, U23.7: now also C50.1, TP3.1
- net at R52.1, R55.1: now also R52.2
- net at R48.2, U19.6 (-), U22.3: now also C41.2
- net at R16.1, R24.2, U11.7: now also C20.1, TP1.1
- net at R40.2, U15.3, U19.2 (-): now also C42.2
- net at U15.6, U17.6 (-): now also R36.3, C33.2; no longer R36.2
- net at R43.1, U19.1: now also C42.1
- net at R41.1, U19.7: now also C41.1
- net at R36.1, R39.1: now also R36.2
- net at R25.1, U10.1: now also C25.1
Other:
- moved on the sheet: C21, C23, C45, C48, R14, R16, R22, R24, R25, R26, R39, R40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

Commit message: Close to final design
Parts:
- R51: renamed from R24; value 22k -> 10k; LCSC PN C31850 -> C25804
- R52: renamed from R39; value 22k -> 10k; LCSC PN C31850 -> C25804
- R53: renamed from R55; value 22k -> 10k; LCSC PN C31850 -> C25804
- R54: renamed from R21; Extended E -> (none); LCSC PN C34846 -> (none)
- R55: renamed from R36; Extended E -> (none); LCSC PN C34846 -> (none)
- R56: renamed from R52; Extended E -> (none); LCSC PN C34846 -> (none)
- U19: renamed from U15; JLCPCB (none) -> 1.88; e14 (none) -> 6.57
- U20: renamed from U9; JLCPCB (none) -> 1.88; e14 (none) -> 6.57
- U21: renamed from U22; JLCPCB (none) -> 1.88; e14 (none) -> 6.57
- renumbered C42 to C29, C25 to C30, C24 to C31, C46 to C32, C49 to C33, C27 to C34, C41 to C35, C33 to C39, C50 to C40, C30 to C41, C31 to C42, C21 to C43, C23 to C44, C48 to C46, C26 to C47, C51 to C48, C28 to C49, C37 to C50, C38 to C51, C20 to C53, R43 to R31, R40 to R32, R48 to R33, R26 to R34, R25 to R35, R17 to R36, R20 to R37, R41 to R38, R19 to R39, R22 to R40, R33 to R41, R35 to R42, R50 to R43, R53 to R44, R30 to R45, R14 to R46, R46 to R47, R16 to R48, R32 to R49, R47 to R50, U10 to U17, U19 to U18, U11 to U23, U17 to U24, U23 to U25
