File: electrical/campervan_management_V2/flow_sensors.kicad_sch (KiCad schematic)
At the start: 8 parts, among them J12 Input Flow Sensor, J13 Output Flow Sensor, U28 LTV-817S-TA1-C, U30 LTV-817S-TA1-C

Commit message: updated 4V1 switcher resistor values. Clean up and reannotate PCB
Parts:
- renumbered C56 to C54, J13 to J10, J12 to J11, R59 to R57, U30 to U26, U28 to U27
Changed lines of the file:
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@@
 		(on_board yes)
 		(dnp no)
-		(property "Reference" "J12"
+		(property "Reference" "J11"
 			(at 75.565 58.42 0)
 			(effects
@@
 			(project "campervan_management_V2"
 				(path "/870a08cc-a6e6-4310-b4b3-ae6af01530aa/37297b33-2fc6-4e16-92e6-9c5c7349d50e"
-					(reference "J12")
+					(reference "J11")
 					(unit 1)
 				)
@@
 		(on_board yes)
 		(dnp no)
-		(property "Reference" "C56"
+		(property "Reference" "C54"
 			(at 121.92 113.0362 0)
 			(effects
@@
 			(project "campervan_management_V2"
 				(path "/870a08cc-a6e6-4310-b4b3-ae6af01530aa/37297b33-2fc6-4e16-92e6-9c5c7349d50e"
-					(reference "C56")
+					(reference "C54")
 					(unit 1)
 				)
@@
 		(on_board yes)
 		(dnp no)
-		(property "Reference" "U30"
+		(property "Reference" "U26"
 			(at 114.3 97.79 0)
 			(effects
@@
 			(project "campervan_management_V2"
 				(path "/870a08cc-a6e6-4310-b4b3-ae6af01530aa/37297b33-2fc6-4e16-92e6-9c5c7349d50e"
-					(reference "U30")
+					(reference "U26")
 					(unit 1)
 				)
@@
 		(on_board yes)
 		(dnp no)
-		(property "Reference" "U28"
+		(property "Reference" "U27"
 			(at 114.3 59.69 0)
 			(effects
@@
 			(project "campervan_management_V2"
 				(path "/870a08cc-a6e6-4310-b4b3-ae6af01530aa/37297b33-2fc6-4e16-92e6-9c5c7349d50e"
-					(reference "U28")
+					(reference "U27")
 					(unit 1)
 				)
@@
 		(on_board yes)
 		(dnp no)
-		(property "Reference" "J13"
+		(property "Reference" "J10"
 			(at 76.835 96.52 0)
 			(effects
@@
 			(project "campervan_management_V2"
 				(path "/870a08cc-a6e6-4310-b4b3-ae6af01530aa/37297b33-2fc6-4e16-92e6-9c5c7349d50e"
-					(reference "J13")
+					(reference "J10")
 					(unit 1)
 				)
@@
 		(dnp no)
 		(fields_autoplaced yes)
-		(property "Reference" "R59"
+		(property "Reference" "R57"
 			(at 97.79 97.79 90)
 			(effects
@@
 			(project "campervan_management_V2"
 				(path "/870a08cc-a6e6-4310-b4b3-ae6af01530aa/37297b33-2fc6-4e16-92e6-9c5c7349d50e"
-					(reference "R59")
-					(unit 1)
-				)
+					(reference "R57")
+					(unit 1)
+				)
